File: src/2022年度回路班_新電源基板.brd (EAGLE design)
At the start: 112.7 x 77 mm, 46 parts

Commit message: ベタの追加
Parts:
- moved JP1 106.9 mm to (2.41, 5.51)
- moved R3 89.8 mm to (7.59, 2.48)
- moved R4 82.8 mm to (15.6, 0.52)
- moved IRLB-3 14.0 mm to (54.0, 59.4), turned to 270 degrees
- moved IRLB-4 14.0 mm to (40.0, 59.4), flipped to the bottom
- moved P-5 5.14 mm to (83.8, 55.0), turned to 90 degrees
- moved P-6 5.14 mm to (83.8, 57.5), turned to 90 degrees
- moved P-7 5.14 mm to (83.8, 60.1), turned to 90 degrees
- moved P-8 5.14 mm to (83.8, 62.6), turned to 90 degrees
- flipped IRLB-1 to the bottom, turned to 270 degrees
Routing:
- net N$22: track 106.6 -> 0.00 mm
- net N$21: track 101.5 -> 18.7 mm
- net N$24: track 52.8 -> 0.00 mm, vias 1 -> 0
- net GND: track 15.8 -> 3.68 mm
- net N$20: track 7.54 -> 0.00 mm
- net N$11: track 2.54 -> 0.00 mm
- net N$7: track 2.54 -> 0.00 mm
- added copper zone on layer 16, net N$12
- added copper zone on layer 1, net N$25
- added copper zone on layer 16, net N$7
- added copper zone on layer 1, net N$8
- removed copper zone on layer 1, net N$12
- removed copper zone on layer 16, net N$25
- removed copper zone on layer 1, net N$7
- removed copper zone on layer 16, net N$8

Commit message: 配線の追加
Parts:
- moved JP1 95.0 mm to (97.4, 7.51)
- moved R3 55.0 mm to (48.2, 39.5)
- moved R4 48.9 mm to (48.2, 36.9)
Routing:
- net VCC2: track 112.3 -> 24.6 mm
- net GND2: track 145.6 -> 60.3 mm
- net N$21: track 18.7 -> 92.6 mm
- net PWM1: track 67.2 -> 13.3 mm
- net N$20: track 0.00 -> 36.2 mm
- net N$22: track 0.00 -> 27.6 mm
- net GND: track 3.68 -> 11.4 mm
- net PWM2: track 45.5 -> 37.9 mm
- net N$19: track 94.1 -> 88.9 mm
- net LED: track 37.7 -> 39.0 mm
- net DIR4: track 25.1 -> 24.5 mm
- net PWM3: track 30.2 -> 29.6 mm

Commit message: 配線の追加
Routing:
- net PWM1: track 13.3 -> 72.0 mm
- net GND2: track 60.3 -> 79.5 mm
- net PWM2: track 37.9 -> 50.2 mm
- net VCC2: track 24.6 -> 33.2 mm, vias 0 -> 1
- net DIR4: track 24.5 -> 25.9 mm, vias 0 -> 1
Changed lines of the file:
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@@
 <wire x1="20.0057" y1="57.7247" x2="20.0057" y2="57.748" width="0.1524" layer="16"/>
 <wire x1="20.0885" y1="57.7247" x2="20.0057" y2="57.7247" width="0.1524" layer="16"/>
-<wire x1="27.83" y1="8.54" x2="20.0885" y2="57.7247" width="0" layer="19" extent="16-16"/>
+<wire x1="23.6932" y1="54.0605" x2="20.0057" y2="57.748" width="0.1524" layer="1"/>
+<wire x1="23.6932" y1="52.32995" x2="23.6932" y2="54.0605" width="0.1524" layer="1"/>
+<wire x1="26.6264" y1="30.74145" x2="26.6264" y2="42.55425" width="0.1524" layer="1"/>
+<wire x1="26.6264" y1="42.55425" x2="29.0336" y2="44.96145" width="0.1524" layer="1"/>
+<wire x1="29.0336" y1="44.96145" x2="29.0336" y2="46.98955" width="0.1524" layer="1"/>
+<wire x1="29.0336" y1="46.98955" x2="23.6932" y2="52.32995" width="0.1524" layer="1"/>
+<wire x1="27.83" y1="8.54" x2="24" y2="12.37" width="0.1524" layer="1"/>
+<wire x1="24" y1="12.37" x2="24" y2="19.61185" width="0.1524" layer="1"/>
+<wire x1="29.1606" y1="24.77245" x2="29.1606" y2="28.20725" width="0.1524" layer="1"/>
+<wire x1="24" y1="19.61185" x2="29.1606" y2="24.77245" width="0.1524" layer="1"/>
+<wire x1="29.1606" y1="28.20725" x2="26.6264" y2="30.74145" width="0.1524" layer="1"/>
 </signal>
 <signal name="PWM2">
@@
 <wire x1="20.0057" y1="60.288" x2="23.998" y2="56.2957" width="0.1524" layer="1"/>
 <wire x1="31.7006" y1="35.1106" x2="27.83" y2="31.24" width="0.1524" layer="1"/>
-<wire x1="31.7006" y1="47.2204" x2="31.7006" y2="35.1106" width="0.1524" layer="1"/>
-<wire x1="23.998" y1="56.2957" x2="23.998" y2="54.923" width="0.1524" layer="1"/>
-<wire x1="31.7006" y1="47.2204" x2="23.998" y2="54.923" width="0" layer="19" extent="1-1"/>
+<wire x1="31.7006" y1="47.2204" x2="31.7006" y2="47" width="0.1524" layer="1"/>
+<wire x1="31.7006" y1="47" x2="31.7006" y2="35.1106" width="0.1524" layer="1"/>
+<wire x1="23.998" y1="56.2957" x2="23.998" y2="55" width="0.1524" layer="1"/>
+<wire x1="23.998" y1="55" x2="23.998" y2="54.923" width="0.1524" layer="1"/>
+<wire x1="23.998" y1="54.923" x2="23.998" y2="52.45620625" width="0.1524" layer="1"/>
+<wire x1="29.5846" y1="49.3364" x2="31.7006" y2="47.2204" width="0.1524" layer="1"/>
+<wire x1="23.998" y1="52.45620625" x2="27.11780625" y2="49.3364" width="0.1524" layer="1"/>
+<wire x1="27.11780625" y1="49.3364" x2="29.5846" y2="49.3364" width="0.1524" layer="1"/>
 </signal>
 <signal name="PWM3">
@@
 <wire x1="48.92" y1="14.81" x2="97.41" y2="8.78" width="0" layer="19" extent="1-1"/>
 <wire x1="52.038" y1="36.902" x2="48.92" y2="14.81" width="0" layer="19" extent="1-1"/>
-<wire x1="48.92" y1="56.81" x2="52.038" y2="36.902" width="0" layer="19" extent="1-1"/>
-<wire x1="8.43" y1="9.89" x2="45.08" y2="14.81" width="0" layer="19" extent="1-1"/>
 </signal>
 <signal name="DIR4">
@@
 <wire x1="14.2283" y1="66.294" x2="15.1543" y2="65.368" width="0.1524" layer="16"/>
 <wire x1="6.199" y1="66.294" x2="14.2283" y2="66.294" width="0.1524" layer="16"/>
-<wire x1="27.83" y1="67.76" x2="21.72044375" y2="67.76" width="0.1524" layer="1"/>
-<wire x1="21.72044375" y1="67.76" x2="20.56669375" y2="66.60625" width="0.1524" layer="1"/>
-<wire x1="16.39255" y1="66.60625" x2="15.1543" y2="65.368" width="0.1524" layer="1"/>
-<wire x1="20.56669375" y1="66.60625" x2="16.39255" y2="66.60625" width="0.1524" layer="1"/>
+<wire x1="15.1543" y1="65.368" x2="16.8953" y2="63.627" width="0.1524" layer="1"/>
+<wire x1="16.8953" y1="63.627" x2="17.272" y2="63.627" width="0.1524" layer="1"/>
+<via x="17.272" y="63.627" extent="1-16" drill="0.35"/>
+<wire x1="17.272" y1="63.627" x2="18.81495625" y2="63.627" width="0.1524" layer="16"/>
+<wire x1="18.81495625" y1="63.627" x2="19.44470625" y2="64.25675" width="0.1524" layer="16"/>
+<wire x1="23.8779125" y1="67.7066" x2="27.7766" y2="67.7066" width="0.1524" layer="16"/>
+<wire x1="19.44470625" y1="64.25675" x2="20.4280625" y2="64.25675" width="0.1524" layer="16"/>
+<wire x1="20.4280625" y1="64.25675" x2="23.8779125" y2="67.7066" width="0.1524" layer="16"/>
+<wire x1="27.7766" y1="67.7066" x2="27.83" y2="67.76" width="0.1524" layer="16"/>
 </signal>
 <signal name="DIR3">
@@
 <wire x1="14.351" y1="58.674" x2="15.1543" y2="57.8707" width="0.1524" layer="16"/>
 <wire x1="15.1543" y1="57.8707" x2="15.1543" y2="57.748" width="0.1524" layer="16"/>
-<wire x1="27.83" y1="3.46" x2="24.13" y2="7.16" width="0.1524" layer="1"/>
+<wire x1="27.83" y1="3.46" x2="23.368" y2="7.922" width="0.1524" layer="1"/>
 <wire x1="15.1543" y1="57.748" x2="15.1543" y2="57.6435875" width="0.1524" layer="1"/>
-<wire x1="24.13" y1="48.6678875" x2="15.1543" y2="57.6435875" width="0.1524" layer="1"/>
-<wire x1="24.13" y1="7.16" x2="24.13" y2="48.6678875" width="0.1524" layer="1"/>
+<wire x1="23.368" y1="49.4298875" x2="15.1543" y2="57.6435875" width="0.1524" layer="1"/>
+<wire x1="23.368" y1="7.922" x2="23.368" y2="49.4298875" width="0.1524" layer="1"/>
 </signal>
 <signal name="LED">
@@
 <wire x1="30.37" y1="73.135" x2="30.37" y2="72.84" width="0.1524" layer="16"/>
 <wire x1="16.4613" y1="69.215" x2="21.463" y2="69.215" width="0.1524" layer="16"/>
-<wire x1="13.18" y1="45.79" x2="30.37" y2="50.54" width="0" layer="19" extent="1-1"/>
-<wire x1="30.37" y1="31.24" x2="30.37" y2="50.54" width="0" layer="19" extent="1-1"/>
+<wire x1="13.18" y1="45.79" x2="16.39" y2="49" width="0.1524" layer="16"/>
+<wire x1="28.83" y1="49" x2="30.37" y2="50.54" width="0.1524" layer="16"/>
+<wire x1="16.39" y1="49" x2="28.83" y2="49" width="0.1524" layer="16"/>
+<wire x1="30.37" y1="50.54" x2="30.37" y2="31.24" width="0" layer="19" extent="1-1"/>
 <wire x1="30.37" y1="8.54" x2="30.37" y2="31.24" width="0" layer="19" extent="1-1"/>
 </signal>
@@
 <wire x1="104.69" y1="10.114" x2="102.916" y2="10.114" width="0.1524" layer="16"/>
 <wire x1="102.916" y1="10.114" x2="101.6" y2="11.43" width="0.1524" layer="16"/>
-<wire x1="101.6" y1="11.43" x2="60.85" y2="8.54" width="0" layer="19" extent="1-1"/>
+<wire x1="60.85" y1="8.54" x2="101.6" y2="11.43" width="0" layer="19" extent="1-1"/>
 </signal>
 <signal name="N$17">
@@
 <wire x1="18.8997" y1="66.802" x2="20.0057" y2="67.908" width="0.1524" layer="16"/>
 <wire x1="8.697" y1="66.802" x2="18.8997" y2="66.802" width="0.1524" layer="16"/>
-<wire x1="30.37" y1="67.76" x2="29.042" y2="69.088" width="0.1524" layer="1"/>
-<wire x1="21.1857" y1="69.088" x2="20.0057" y2="67.908" width="0.1524" layer="1"/>
-<wire x1="29.042" y1="69.088" x2="21.1857" y2="69.088" width="0.1524" layer="1"/>
-<wire x1="30.37" y1="45.46" x2="30.37" y2="67.76" width="0" layer="19" extent="1-1"/>
+<wire x1="20.0057" y1="67.908" x2="18.034" y2="65.9363" width="0.1524" layer="1"/>
+<wire x1="18.034" y1="65.9363" x2="18.034" y2="62.992" width="0.1524" layer="1"/>
+<via x="18.034" y="62.992" extent="1-16" drill="0.35"/>
+<wire x1="18.034" y1="62.992" x2="18.3642" y2="63.3222" width="0.1524" layer="16"/>
+<wire x1="18.3642" y1="63.3222" x2="18.9412125" y2="63.3222" width="0.1524" layer="16"/>
+<wire x1="19.5709625" y1="63.95195" x2="20.55431875" y2="63.95195" width="0.1524" layer="16"/>
+<wire x1="23.02336875" y1="66.421" x2="29.083" y2="66.421" width="0.1524" layer="16"/>
+<wire x1="18.9412125" y1="63.3222" x2="19.5709625" y2="63.95195" width="0.1524" layer="16"/>
+<wire x1="20.55431875" y1="63.95195" x2="23.02336875" y2="66.421" width="0.1524" layer="16"/>
+<wire x1="29.083" y1="66.421" x2="30.37" y2="67.708" width="0.1524" layer="16"/>
+<wire x1="30.37" y1="67.708" x2="30.37" y2="67.76" width="0.1524" layer="16"/>
+<wire x1="30.37" y1="45.46" x2="18.034" y2="62.992" width="0" layer="19" extent="1-1"/>
 <wire x1="30.37" y1="26.16" x2="30.37" y2="45.46" width="0" layer="19" extent="1-1"/>
 <wire x1="30.37" y1="3.46" x2="30.37" y2="26.16" width="0" layer="19" extent="1-1"/>
@@
 <polygon width="0.1524" layer="16" thermals="no">
 <vertex x="89" y="58.492"/>
-<vertex x="38.327" y="58.492"/>
-<vertex x="38.327" y="52.619"/>
-<vertex x="32" y="52.619"/>
+<vertex x="51.327" y="58.492"/>
+<vertex x="51.327" y="48.619"/>
+<vertex x="32" y="48.619"/>
 <vertex x="32" y="44"/>
 <vertex x="62" y="44"/>
