File: src/2022年度回路班_新電源基板.brd (EAGLE design)
At the start: 112.7 x 77 mm, 46 parts

Commit message: 配線の追加
Parts:
- moved JP1 95.0 mm to (97.4, 7.51)
- moved R3 55.0 mm to (48.2, 39.5)
- moved R4 48.9 mm to (48.2, 36.9)
Routing:
- net VCC2: track 112.3 -> 33.2 mm, vias 0 -> 1
- net N$21: track 18.7 -> 92.6 mm
- net GND2: track 145.6 -> 79.3 mm
- net N$20: track 0.00 -> 36.2 mm
- net N$22: track 0.00 -> 27.6 mm
- net GND: track 3.68 -> 11.4 mm
- net N$19: track 94.1 -> 88.9 mm
- net PWM1: track 67.2 -> 72.0 mm
- net PWM2: track 45.5 -> 50.2 mm
- net LED: track 37.7 -> 39.0 mm
- net DIR4: track 25.1 -> 25.9 mm, vias 0 -> 1
- net PWM3: track 30.2 -> 29.6 mm

Commit message: 配線の追加
Parts:
- moved IRLB-1 0.22 mm to (40.0, 17.6)
- moved IRLB-2 0.22 mm to (54.0, 17.6)
- moved IRLB-3 0.11 mm to (54.0, 59.2)
- moved IRLB-4 0.11 mm to (40.0, 59.2)
Routing:
- net VCC: track 3.64 -> 103.8 mm
- net N$24: track 0.00 -> 81.1 mm, vias 0 -> 1
- net VCC2: track 33.2 -> 106.1 mm
- net GND: track 11.4 -> 62.3 mm
- net N$20: track 36.2 -> 86.6 mm
- net GND2: track 79.3 -> 128.3 mm
- net N$22: track 27.6 -> 51.1 mm
- net N$19: track 88.9 -> 93.5 mm
- net PWM1: track 72.0 -> 72.7 mm

Commit message: DRCエラーの解消
Routing:
- net GND: track 62.3 -> 61.3 mm
- net PWM3: track 29.6 -> 30.1 mm
Changed lines of the file:
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@@
 <wire x1="18.923" y1="56.642" x2="20.0057" y2="57.7247" width="0.1524" layer="16"/>
 <wire x1="20.0057" y1="57.7247" x2="20.0057" y2="57.748" width="0.1524" layer="16"/>
-<wire x1="20.0885" y1="57.7247" x2="20.0057" y2="57.7247" width="0.1524" layer="16"/>
 <wire x1="23.1852" y1="54.5685" x2="20.0057" y2="57.748" width="0.1524" layer="1"/>
 <wire x1="23.1852" y1="52.07595" x2="23.1852" y2="54.5685" width="0.1524" layer="1"/>
@@
 <contactref element="EDGE3" pad="P$25"/>
 <wire x1="7.702" y1="62.717" x2="8.697" y2="61.722" width="0.1524" layer="16"/>
-<wire x1="18.8997" y1="61.722" x2="20.0057" y2="62.828" width="0.1524" layer="16"/>
 <wire x1="8.697" y1="61.722" x2="18.8997" y2="61.722" width="0.1524" layer="16"/>
-<wire x1="20.0057" y1="62.828" x2="20.0057" y2="62.7983" width="0.1524" layer="16"/>
-<wire x1="24.3028" y1="52.5824625" x2="24.3028" y2="58.5309" width="0.1524" layer="1"/>
-<wire x1="24.3028" y1="58.5309" x2="20.0057" y2="62.828" width="0.1524" layer="1"/>
+<wire x1="24.3028" y1="52.5824625" x2="24.3028" y2="58" width="0.1524" layer="1"/>
+<wire x1="24.3028" y1="58" x2="24.3028" y2="58.5309" width="0.1524" layer="1"/>
 <wire x1="27.83" y1="50.54" x2="26.3452625" y2="50.54" width="0.1524" layer="1"/>
 <wire x1="26.3452625" y1="50.54" x2="24.3028" y2="52.5824625" width="0.1524" layer="1"/>
+<wire x1="24.3028" y1="58" x2="20.0057" y2="62.2971" width="0.1524" layer="1"/>
+<wire x1="20.0057" y1="62.2971" x2="20.0057" y2="62.828" width="0.1524" layer="1"/>
+<wire x1="18.8997" y1="61.722" x2="20.0057" y2="62.828" width="0.1524" layer="16"/>
 </signal>
 <signal name="PWM4">
@@
 <wire x1="106.09" y1="10.114" x2="104.756" y2="8.78" width="0.1524" layer="16"/>
 <wire x1="104.756" y1="8.78" x2="97.41" y2="8.78" width="0.1524" layer="16"/>
-<wire x1="109.22" y1="11.43" x2="109.22" y2="11.5217125" width="0.1524" layer="16"/>
-<wire x1="109.22" y1="11.5217125" x2="111.303" y2="13.6047125" width="0.1524" layer="16"/>
-<wire x1="111.303" y1="13.6047125" x2="111.303" y2="60" width="0.1524" layer="16"/>
+<wire x1="111.303" y1="13.4777125" x2="109.2552875" y2="11.43" width="0.1524" layer="16"/>
+<wire x1="109.22" y1="11.43" x2="109.2552875" y2="11.43" width="0.1524" layer="16"/>
+<wire x1="111.303" y1="13.4777125" x2="111.303" y2="58.984" width="0.1524" layer="16"/>
 </signal>
 <signal name="DIR4">
@@
 <wire x1="100.37" y1="63.15" x2="108.37" y2="63.15" width="0.1524" layer="16"/>
 <wire x1="108.37" y1="63.15" x2="110" y2="64.78" width="0.1524" layer="16"/>
-<wire x1="110" y1="64.78" x2="110" y2="71" width="0.1524" layer="16"/>
+<wire x1="110" y1="64.78" x2="110" y2="64.907" width="0.1524" layer="16"/>
+<wire x1="110" y1="64.653" x2="110" y2="64.78" width="0.1524" layer="16"/>
+<wire x1="110" y1="64.907" x2="110" y2="71" width="0.1524" layer="16"/>
 <wire x1="110" y1="71" x2="108.91" y2="72.09" width="0.1524" layer="16"/>
 <wire x1="108.91" y1="72.09" x2="108.37" y2="72.09" width="0.1524" layer="16"/>
-<wire x1="110" y1="64.78" x2="111.6078" y2="63.1722" width="0.1524" layer="16"/>
-<wire x1="111.6078" y1="63.1722" x2="111.6078" y2="8.635" width="0.1524" layer="16"/>
+<wire x1="110" y1="64.653" x2="111.6078" y2="63.0452" width="0.1524" layer="16"/>
+<wire x1="111.6078" y1="63.0452" x2="111.6078" y2="8.635" width="0.1524" layer="16"/>
 <wire x1="111.6078" y1="8.635" x2="106.7828" y2="3.81" width="0.1524" layer="16"/>
 <wire x1="106.7828" y1="3.81" x2="106.68" y2="3.81" width="0.1524" layer="16"/>
