File: src/2022年度回路班_新電源基板.sch (EAGLE design)
At the start: 54 parts, among them P1 RUEF900-2, P10 RUEF900-2, P11 RUEF900-2, P12 RUEF900-2, P13 RUEF900-2, P14 RUEF900-2, P15 RUEF900-2, P16 RUEF900-2, P2 RUEF900-2, P3 RUEF900-2, P4 RUEF900-2, P5 RUEF900-2, P6 RUEF900-2, P7 RUEF900-2, P8 RUEF900-2, P9 RUEF900-2

Commit message: 部品の配置
Parts:
- removed P1, P10, P11, P12, P13, P14, P15, P16, P2, P3, P4, P5, P6, P7, P8, P9: RUEF900-2, RUEF900-2:RUEF900-2
- added P-1, P-2, P-3, P-4, P-5, P-6, P-7, P-8: P-SWITCH, OKUDA_libraries:P-SWITCH
Connections:
- net N$11: now also P-3.P$2, P-4.P$2; no longer P5.1, P6.1, P7.1, P8.1
- net N$12: now also P-7.P$2, P-8.P$2; no longer P13.1, P14.1, P15.1, P16.1
- net N$15: now also P-5.P$2, P-6.P$2; no longer P10.1, P11.1, P12.1, P9.1
- net N$16: now also P-7.P$1, P-8.P$1; no longer P13.2, P14.2, P15.2, P16.2
- net N$23: now also P-5.P$1, P-6.P$1; no longer P10.2, P11.2, P12.2, P9.2
- net N$25: now also P-1.P$1, P-2.P$1; no longer P1.2, P2.2, P3.2, P4.2
- net N$7: now also P-1.P$2, P-2.P$2; no longer P1.1, P2.1, P3.1, P4.1
- net N$8: now also P-3.P$1, P-4.P$1; no longer P5.2, P6.2, P7.2, P8.2

Commit message: 配線の追加
Connections:
- removed net N$16: EDGE4.P18, EDGE4.P19, EDGE4.P20, EDGE4.P21, EDGE4.P22, EDGE4.P23, EDGE4.P28, EDGE4.P29, EDGE4.P30, EDGE4.P31, EDGE4.P32, EDGE4.P33, P-7.P$1, P-8.P$1
- removed net N$23: EDGE3.P18, EDGE3.P19, EDGE3.P20, EDGE3.P21, EDGE3.P22, EDGE3.P23, EDGE3.P28, EDGE3.P29, EDGE3.P30, EDGE3.P31, EDGE3.P32, EDGE3.P33, P-5.P$1, P-6.P$1
- new net N$14: EDGE3.P28, EDGE3.P29, EDGE3.P30, EDGE3.P31, EDGE3.P32, EDGE3.P33, EDGE3.P34, EDGE3.P35, EDGE3.P36, EDGE3.P37, EDGE3.P38, EDGE3.P39, P-5.P$1, P-6.P$1
- new net N$26: EDGE2.P28, EDGE2.P29, EDGE2.P30, EDGE2.P31, EDGE2.P32, EDGE2.P33, EDGE2.P34, EDGE2.P35, EDGE2.P36, EDGE2.P37, EDGE2.P38, EDGE2.P39, P-3.P$1, P-4.P$1
- net N$25: now also EDGE1.P34, EDGE1.P35, EDGE1.P36, EDGE1.P37, EDGE1.P38, EDGE1.P39; no longer EDGE1.P18, EDGE1.P19, EDGE1.P20, EDGE1.P21, EDGE1.P22, EDGE1.P23
- net N$8: now also EDGE4.P28, EDGE4.P29, EDGE4.P30, EDGE4.P31, EDGE4.P32, EDGE4.P33, EDGE4.P34, EDGE4.P35, EDGE4.P36, EDGE4.P37, EDGE4.P38, EDGE4.P39, P-7.P$1, P-8.P$1; no longer EDGE2.P18, EDGE2.P19, EDGE2.P20, EDGE2.P21, EDGE2.P22, EDGE2.P23, EDGE2.P28, EDGE2.P29, EDGE2.P30, EDGE2.P31, EDGE2.P32, EDGE2.P33, P-3.P$1, P-4.P$1
- net VCC: now also EDGE1.P18, EDGE1.P19, EDGE1.P20, EDGE1.P21, EDGE1.P22, EDGE1.P23, EDGE2.P18, EDGE2.P19, EDGE2.P20, EDGE2.P21, EDGE2.P22, EDGE2.P23, EDGE3.P18, EDGE3.P19, EDGE3.P20, EDGE3.P21, EDGE3.P22, EDGE3.P23, EDGE4.P18, EDGE4.P19, EDGE4.P20, EDGE4.P21, EDGE4.P22, EDGE4.P23; no longer EDGE1.P34, EDGE1.P35, EDGE1.P36, EDGE1.P37, EDGE1.P38, EDGE1.P39, EDGE2.P34, EDGE2.P35, EDGE2.P36, EDGE2.P37, EDGE2.P38, EDGE2.P39, EDGE3.P34, EDGE3.P35, EDGE3.P36, EDGE3.P37, EDGE3.P38, EDGE3.P39, EDGE4.P34, EDGE4.P35, EDGE4.P36, EDGE4.P37, EDGE4.P38, EDGE4.P39
