File: src/2022年度回路班_新電源基板.kicad_pcb (KiCad board)
At the start: 2 copper layers, 112.7 x 77 mm, 47 parts

Commit message: QRコードの拡大
Parts:
- removed the G*** at (104.3, 133.5)
- added G***: LOGO, 2022年度回路班_新電源基板:電源基板QRコード_拡大版, B.Cu at (103.8, 132.9)
