File: src/2022年度回路班_新電源基板.kicad_pcb (KiCad board)
At the start: 2 copper layers, 112.7 x 77 mm, 51 parts

Commit message: エラーの解消
Parts:
- moved G*** 0.34 mm to (105.7, 133.5)
Other:
- board text added: "B series"
- board text added: "PowerUnit"
- board text added: "ver 1.0"

Commit message: 基板デザインの完成
Parts:
- added G***: LOGO, 2022年度回路班_新電源基板:メカテック部ロゴ_縮小, B.Cu at (124.5, 105.3)
Other:
- board text added: "IN"
- board text added: "MDC"
- board text added: "POW"
