File: src/PowerUnit-Bseries(ver1.0).kicad_pcb (KiCad board)
At the start: 2 copper layers, 112.7 x 77 mm, 50 parts

Commit message: 基盤デザインの完成 gerber出力
Parts:
- added G***: LOGO, PowerUnit-Bseries(ver1.0):メカテック部ロゴ_縮小, B.Cu at (128.1, 104.8)
- added G***: LOGO, PowerUnit-Bseries(ver1.0):電源基板QRコード_拡大版, B.Cu at (109.5, 134.2)
- moved R3 2.70 mm to (143.1, 103.7)
- moved R4 2.68 mm to (143.1, 106.5)
Routing:
- net GND: track 111.6 -> 114.4 mm
- net Net-(R3-Pad1): track 96.6 -> 93.8 mm
- net Net-(IRLB-1-PadG): track 65.2 -> 67.9 mm
Other:
- board text added: "B series"
- board text added: "PowerUnit"
