File: src/(Eagle)PowerUnit-Bseries(ver1.0).brd (EAGLE design)
At the start: 100 x 80 mm, 51 parts

Commit message: XT60PWコネクタに変えた
Parts:
- removed IN+, IN-, OUT1+, OUT1-, OUT2+, OUT2-, OUT3+, OUT3-, THRU+, THRU-: PADS14, OKUDA_libraries:AWG14
- added CON1: XT90PW-M, amass:XT90PW-M
- added CON2: XT90PW-F, amass:XT90PW-F
- added CON3, CON4, CON5, CON6: XT60PW-F, amass:XT60PW-F
- added U1: LQFP64, STM32F446xC:STM32F446XC
- added U2: MCP2517FD, MCP2517FD:MCP2517FD
- H1, H2, H3, H4: value MOUNT-HOLE3.2 -> MOUNT-HOLE3.2(NORESIST); device holes:3,2 -> MOUNT-HOLE3.2(NORESIST):3,2
- moved H4 147.5 mm to (-146.1, -40.6)
- moved H3 143.8 mm to (-146.1, -33.0)
- moved H2 141.0 mm to (-146.1, -25.4)
- moved H1 139.1 mm to (-146.1, -17.8)
Connections:
- new net +: CON5.+, CON6.+
- new net -: CON5.-, CON6.-
- net GND: now also CON1.-, CON2.-, H1.P$1, H2.P$1, H3.P$1, H4.P$1; no longer IN-.P$1, THRU-.P$1
- net N$1: now also CON3.-; no longer OUT1-.P$1
- net N$2: now also CON4.-; no longer OUT2-.P$1
- net N$4: now also CON3.+; no longer OUT1+.P$1
- net N$5: now also CON4.+; no longer OUT2+.P$1
- net N$6: no longer OUT3+.P$1
- net N$9: no longer OUT3-.P$1
- net VCC: now also CON1.+, CON2.+; no longer IN+.P$1, THRU+.P$1
Other:
- board size 100 x 80 mm -> 100 x 100 mm

Commit message: トランシーバ選定途中、XT60PW
Parts:
- removed EDGE5: 7-5530843-6, 7-5530843-6:7-5530843-6
- removed OUT4+, OUT4-: PADS14, OKUDA_libraries:AWG14
- moved CON6 309.5 mm to (72.4, 83.8)
- moved CON5 276.0 mm to (53.3, 83.8)
- moved CON4 243.5 mm to (34.3, 83.8)
- moved CON3 212.5 mm to (15.2, 83.8)
- moved EDGE4 95.3 mm to (-143.5, 71.1), turned to 90 degrees
Connections:
- removed net +: CON5.+, CON6.+
- removed net -: CON5.-, CON6.-
- removed net NC: EDGE5.P$7
- net DIR1: no longer EDGE5.P$12
- net DIR2: no longer EDGE5.P$11
- net DIR3: no longer EDGE5.P$10
- net DIR4: no longer EDGE5.P$9
- net GND2: no longer EDGE5.P$8
- net LED: no longer EDGE5.P$6
- net N$10: now also CON6.+; no longer OUT4+.P$1
- net N$13: now also CON6.-; no longer OUT4-.P$1
- net N$6: now also CON5.+
- net N$9: now also CON5.-
- net PWM1: no longer EDGE5.P$1
- net PWM2: no longer EDGE5.P$2
- net PWM3: no longer EDGE5.P$3
- net PWM4: no longer EDGE5.P$4
- net VCC2: no longer EDGE5.P$5

Commit message: CANトランシーバの選定(クリスマスイブですよ？（笑）)
Parts:
- added U$1: MCP2558FD, MCP2558FD:MCP2558FD
Connections:
- net GND: now also U2.VSS
Changed lines of the file:
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@@
 <attribute name="VALUE" x="67.39" y="99.12" size="1.778" layer="27"/>
+</element>
+<element name="U$1" library="MCP2558FD" package="MCP2558FD" package3d_urn="urn:adsk.eagle:package:38673258/1" value="MCP2558FD" x="64.77" y="8.89" smashed="yes">
+<attribute name="VALUE" x="63.57" y="7.89" size="0.381" layer="27" rot="R90"/>
 </element>
 </elements>
@@
 <contactref element="H3" pad="P$1"/>
 <contactref element="H4" pad="P$1"/>
+<contactref element="U2" pad="VSS"/>
 <wire x1="-146.05" y1="-33.02" x2="-146.05" y2="-40.64" width="0" layer="19" extent="1-1"/>
 <wire x1="-146.05" y1="-25.4" x2="-146.05" y2="-33.02" width="0" layer="19" extent="1-1"/>
 <wire x1="-146.05" y1="-17.78" x2="-146.05" y2="-25.4" width="0" layer="19" extent="1-1"/>
-<wire x1="37.73" y1="22.86" x2="-146.05" y2="-17.78" width="0" layer="19" extent="1-1"/>
-<wire x1="24.5" y1="22.86" x2="37.73" y2="22.86" width="0" layer="19" extent="1-1"/>
-<wire x1="-87.57" y1="8.89" x2="24.5" y2="22.86" width="0" layer="19" extent="1-1"/>
+<wire x1="-87.57" y1="8.89" x2="-146.05" y2="-17.78" width="0" layer="19" extent="1-1"/>
 <wire x1="-96.52" y1="33.02" x2="-87.57" y2="8.89" width="0" layer="19" extent="1-1"/>
 <wire x1="-62.23" y1="2.54" x2="-87.57" y2="8.89" width="0" layer="19" extent="1-1"/>
@@
 <wire x1="-31.75" y1="2.54" x2="-46.99" y2="2.54" width="0" layer="19" extent="1-1"/>
 <wire x1="-16.51" y1="2.54" x2="-31.75" y2="2.54" width="0" layer="19" extent="1-1"/>
+<wire x1="24.5" y1="22.86" x2="-16.51" y2="2.54" width="0" layer="19" extent="1-1"/>
+<wire x1="37.73" y1="22.86" x2="24.5" y2="22.86" width="0" layer="19" extent="1-1"/>
+<wire x1="62.23" y1="6.35" x2="37.73" y2="22.86" width="0" layer="19" extent="1-1"/>
 <wire x1="-88.9" y1="104.14" x2="-96.52" y2="33.02" width="0" layer="19" extent="1-1"/>
 <wire x1="-54.61" y1="104.14" x2="-88.9" y2="104.14" width="0" layer="19" extent="1-1"/>

Commit message: CAN周りの配線など
Parts:
- removed SV1: (no value), con-ml:ML10
- added JP2: (no value), pinhead:1X02
- added R7: 120Ω, CR0603:CR0603
- added USB1: 5077CR-16SMC2-BK-TR, 5077CR-16SMC2-BK-TR:5077CR-16SMC2-BK-TR
- moved H1 237.8 mm to (80.0, 55.9)
- moved H2 237.8 mm to (80.0, 48.3)
- moved H3 237.8 mm to (80.0, 40.6)
- moved H4 237.8 mm to (80.0, 33.0)
- moved U1 40.5 mm to (43.2, 53.3)
- moved U$1 38.8 mm to (44.5, 41.9)
- moved U2 37.7 mm to (34.3, 38.1)
Connections:
- new net +5V: USB1.VBUS1, USB1.VBUS2
- new net CANH: R7.RIGHT, U$1.CANH
- new net CANL: JP2.2, U$1.CANL
- new net N$23: JP2.1, R7.LEFT
- new net N$27: U$1.TXD, U2.TXCAN
- new net N$28: U$1.RXD, U2.RXCAN
- net DIR1: no longer SV1.9
- net DIR2: no longer SV1.7
- net DIR3: no longer SV1.5
- net DIR4: no longer SV1.3
- net GND: now also U$1.EP, U$1.VSS, USB1.GND1, USB1.GND2, USB1.SHIELD1, USB1.SHIELD2, USB1.SHIELD3, USB1.SHIELD4
- net GND2: no longer SV1.1
- net PWM1: no longer SV1.10
- net PWM2: no longer SV1.8
- net PWM3: no longer SV1.6
- net PWM4: no longer SV1.4
- net VCC2: no longer SV1.2

Commit message: レギュレータの追加など
Parts:
- added R8, R9: (no value), CR0603:CR0603
- added U3: CH340E, CH340E:MSOP-10
- added U4: AP63203WU-7, AP63203WU-7:AP63203WU-7
- moved R7 164.8 mm to (12.7, 31.8)
Connections:
- new net N$29: R8.RIGHT, USB1.CC2
- new net N$30: R9.RIGHT, USB1.CC1
- new net N$31: U3.UD+, USB1.DP1, USB1.DP2
- new net N$32: U3.UD-, USB1.DN1, USB1.DN2
- net GND: no longer USB1.GND1, USB1.GND2, USB1.SHIELD1, USB1.SHIELD2, USB1.SHIELD3, USB1.SHIELD4
- net GND2: now also R8.LEFT, R9.LEFT, U3.GND, U4.GND, USB1.GND1, USB1.GND2, USB1.SHIELD1, USB1.SHIELD2, USB1.SHIELD3, USB1.SHIELD4
Changed lines of the file:
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@@
 <attribute name="VALUE" x="51.61" y="43.9" size="1" layer="27"/>
 </element>
-<element name="R7" library="CR0603" package="CR0603" value="120Ω" x="-147.32" y="-7.62" smashed="yes">
-<attribute name="VALUE" x="-148.62" y="-6.92" size="0.5" layer="27"/>
+<element name="R7" library="CR0603" package="CR0603" value="120Ω" x="12.7" y="31.75" smashed="yes">
+<attribute name="VALUE" x="11.4" y="32.45" size="0.5" layer="27"/>
+</element>
+<element name="R8" library="CR0603" package="CR0603" value="" x="12.7" y="29.21" smashed="yes">
+<attribute name="VALUE" x="11.4" y="29.91" size="0.5" layer="27"/>
+</element>
+<element name="R9" library="CR0603" package="CR0603" value="" x="12.7" y="26.67" smashed="yes">
+<attribute name="VALUE" x="11.4" y="27.37" size="0.5" layer="27"/>
+</element>
+<element name="U3" library="CH340E" package="MSOP-10" value="CH340E" x="54.61" y="49.53" smashed="yes">
+<attribute name="VALUE" x="52.71" y="47.73" size="0.7" layer="27" rot="R90"/>
+</element>
+<element name="U4" library="AP63203WU-7" package="AP63203WU-7" value="AP63203WU-7" x="40.64" y="33.02" smashed="yes">
+<attribute name="VALUE" x="38.84" y="31.72" size="0.5" layer="27" rot="R90"/>
 </element>
 </elements>
@@
 <contactref element="U$1" pad="VSS"/>
 <contactref element="U2" pad="VSS"/>
-<contactref element="USB1" pad="SHIELD2"/>
-<contactref element="USB1" pad="SHIELD4"/>
-<contactref element="USB1" pad="SHIELD1"/>
-<contactref element="USB1" pad="SHIELD3"/>
-<contactref element="USB1" pad="GND2"/>
-<contactref element="USB1" pad="GND1"/>
 <wire x1="80.01" y1="48.26" x2="80.01" y2="55.88" width="0" layer="19" extent="1-1"/>
 <wire x1="80.01" y1="40.64" x2="80.01" y2="48.26" width="0" layer="19" extent="1-1"/>
 <wire x1="80.01" y1="33.02" x2="80.01" y2="40.64" width="0" layer="19" extent="1-1"/>
-<wire x1="58.93" y1="42.28" x2="80.01" y2="40.64" width="0" layer="19" extent="1-1"/>
-<wire x1="57.81" y1="42.84" x2="58.93" y2="42.28" width="0" layer="19" extent="1-1"/>
-<wire x1="58.93" y1="38.1" x2="58.93" y2="42.28" width="0" layer="19" extent="1-1"/>
-<wire x1="51.41" y1="42.84" x2="57.81" y2="42.84" width="0" layer="19" extent="1-1"/>
-<wire x1="50.29" y1="42.28" x2="51.41" y2="42.84" width="0" layer="19" extent="1-1"/>
-<wire x1="50.29" y1="38.1" x2="50.29" y2="42.28" width="0" layer="19" extent="1-1"/>
-<wire x1="44.45" y1="41.91" x2="50.29" y2="42.28" width="0" layer="19" extent="1-1"/>
+<wire x1="44.45" y1="41.91" x2="80.01" y2="40.64" width="0" layer="19" extent="1-1"/>
 <wire x1="44.2" y1="40.46" x2="44.45" y2="41.91" width="0" layer="19" extent="1-1"/>
 <wire x1="41.91" y1="38.1" x2="44.2" y2="40.46" width="0" layer="19" extent="1-1"/>
@@
 <contactref element="EDGE3" pad="P$24"/>
 <contactref element="EDGE4" pad="P$24"/>
+<contactref element="USB1" pad="SHIELD4"/>
+<contactref element="USB1" pad="SHIELD3"/>
+<contactref element="USB1" pad="SHIELD1"/>
+<contactref element="USB1" pad="SHIELD2"/>
+<contactref element="USB1" pad="GND1"/>
+<contactref element="USB1" pad="GND2"/>
+<contactref element="U3" pad="GND"/>
+<contactref element="R9" pad="LEFT"/>
+<contactref element="R8" pad="LEFT"/>
+<contactref element="U4" pad="GND"/>
+<wire x1="11.7" y1="29.21" x2="11.7" y2="26.67" width="0" layer="19" extent="1-1"/>
+<wire x1="-140.97" y1="99.06" x2="11.7" y2="29.21" width="0" layer="19" extent="1-1"/>
+<wire x1="-33.02" y1="105.41" x2="-140.97" y2="99.06" width="0" layer="19" extent="1-1"/>
 <wire x1="-20.32" y1="60.96" x2="-33.02" y2="105.41" width="0" layer="19" extent="1-1"/>
 <wire x1="-20.32" y1="49.53" x2="-20.32" y2="60.96" width="0" layer="19" extent="1-1"/>
 <wire x1="-20.32" y1="38.1" x2="-20.32" y2="49.53" width="0" layer="19" extent="1-1"/>
-<wire x1="-140.97" y1="99.06" x2="-33.02" y2="105.41" width="0" layer="19" extent="1-1"/>
+<wire x1="41.59" y1="34.1195" x2="-20.32" y2="38.1" width="0" layer="19" extent="1-1"/>
+<wire x1="50.29" y1="38.1" x2="41.59" y2="34.1195" width="0" layer="19" extent="1-1"/>
+<wire x1="50.29" y1="42.28" x2="50.29" y2="38.1" width="0" layer="19" extent="1-1"/>
+<wire x1="51.41" y1="42.84" x2="50.29" y2="42.28" width="0" layer="19" extent="1-1"/>
+<wire x1="54.61" y1="47.555" x2="51.41" y2="42.84" width="0" layer="19" extent="1-1"/>
+<wire x1="57.81" y1="42.84" x2="54.61" y2="47.555" width="0" layer="19" extent="1-1"/>
+<wire x1="58.93" y1="42.28" x2="57.81" y2="42.84" width="0" layer="19" extent="1-1"/>
+<wire x1="58.93" y1="38.1" x2="58.93" y2="42.28" width="0" layer="19" extent="1-1"/>
 </signal>
 <signal name="VCC">
@@
 <contactref element="U$1" pad="CANH"/>
 <contactref element="R7" pad="RIGHT"/>
-<wire x1="44.2" y1="43.36" x2="-146.32" y2="-7.62" width="0" layer="19" extent="1-1"/>
+<wire x1="44.2" y1="43.36" x2="13.7" y2="31.75" width="0" layer="19" extent="1-1"/>
 </signal>
 <signal name="CANL">
@@
 <contactref element="JP2" pad="1"/>
 <contactref element="R7" pad="LEFT"/>
-<wire x1="76.2" y1="25.4" x2="-148.32" y2="-7.62" width="0" layer="19" extent="1-1"/>
+<wire x1="76.2" y1="25.4" x2="11.7" y2="31.75" width="0" layer="19" extent="1-1"/>
 </signal>
 <signal name="N$27">
@@
 <wire x1="52.21" y1="42.84" x2="57.01" y2="42.84" width="0" layer="19" extent="1-1"/>
 </signal>
+<signal name="N$29">
+<contactref element="USB1" pad="CC2"/>
+<contactref element="R8" pad="RIGHT"/>
+<wire x1="56.36" y1="42.84" x2="13.7" y2="29.21" width="0" layer="19" extent="1-1"/>
+</signal>
+<signal name="N$30">
+<contactref element="USB1" pad="CC1"/>
+<contactref element="R9" pad="RIGHT"/>
+<wire x1="53.36" y1="42.84" x2="13.7" y2="26.67" width="0" layer="19" extent="1-1"/>
+</signal>
+<signal name="N$31">
+<contactref element="USB1" pad="DP1"/>
+<contactref element="USB1" pad="DP2"/>
+<contactref element="U3" pad="UD+"/>
+<wire x1="54.36" y1="42.84" x2="53.61" y2="47.555" width="0" layer="19" extent="1-1"/>
+<wire x1="55.36" y1="42.84" x2="54.36" y2="42.84" width="0" layer="19" extent="1-1"/>
+</signal>
+<signal name="N$32">
+<contactref element="USB1" pad="DN1"/>
+<contactref element="USB1" pad="DN2"/>
+<contactref element="U3" pad="UD-"/>
+<wire x1="53.86" y1="42.84" x2="54.11" y2="47.555" width="0" layer="19" extent="1-1"/>
+<wire x1="54.86" y1="42.84" x2="53.86" y2="42.84" width="0" layer="19" extent="1-1"/>
+</signal>
 </signals>

Commit message: 5Vレギュレータの追加など
Parts:
- added C3: GCM188L81H104KA57, GCM188L81H104K57(0.1uF):GCM188L81H104KA57
- added ECHO: (no value), pinhead:1X02
- added LED4: SMLE13BC8T, SML-E12V8WT86:SML-E12V8WT86
- added R10: 150Ω, CR0603:CR0603
- added U5: AP63205WU-7, AP63205WU-7:AP63203WU-7
Connections:
- net +5V renamed U5V
- new net +3V3: C3.P$2, U3.3V3, U3.VCC
- new net N$33: R10.RIGHT, U3.TNOW
- new net N$34: LED4.A, R10.LEFT
- new net USART_RX: ECHO.1, U1.P17, U3.TXD
- new net USART_TX: ECHO.2, U1.P16, U3.RXD
- net GND2: now also C3.P$1, LED4.K, U5.GND
Changed lines of the file:
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@@
 <attribute name="VALUE" x="38.84" y="31.72" size="0.5" layer="27" rot="R90"/>
+</element>
+<element name="U5" library="AP63205WU-7" package="AP63203WU-7" value="AP63205WU-7" x="25.4" y="55.88" smashed="yes">
+<attribute name="VALUE" x="23.6" y="54.58" size="0.5" layer="27" rot="R90"/>
+</element>
+<element name="ECHO" library="pinhead" library_urn="urn:adsk.eagle:library:325" package="1X02" package3d_urn="urn:adsk.eagle:package:22435/2" value="" x="26.67" y="49.53" smashed="yes">
+<attribute name="NAME" x="24.0538" y="51.3588" size="1.27" layer="25" ratio="10"/>
+<attribute name="POPULARITY" value="98" x="26.67" y="49.53" size="1.778" layer="27" display="off"/>
+<attribute name="VALUE" x="24.13" y="46.355" size="1.27" layer="27"/>
+</element>
+<element name="C3" library="GCM188L81H104K57(0.1uF)" package="GCM188L81H104KA57" value="GCM188L81H104KA57" x="24.13" y="45.72" smashed="yes">
+<attribute name="NAME" x="23.33" y="46.22" size="0.1" layer="21"/>
+</element>
+<element name="R10" library="CR0603" package="CR0603" value="150Ω" x="25.4" y="43.18" smashed="yes">
+<attribute name="VALUE" x="24.1" y="43.88" size="0.5" layer="27"/>
+</element>
+<element name="LED4" library="SML-E12V8WT86" package="SML-E12V8WT86" value="SMLE13BC8T" x="21.59" y="43.18" smashed="yes">
+<attribute name="NAME" x="20.955" y="43.688" size="0.127" layer="25" rot="R90"/>
 </element>
 </elements>
@@
 <contactref element="R8" pad="LEFT"/>
 <contactref element="U4" pad="GND"/>
-<wire x1="11.7" y1="29.21" x2="11.7" y2="26.67" width="0" layer="19" extent="1-1"/>
-<wire x1="-140.97" y1="99.06" x2="11.7" y2="29.21" width="0" layer="19" extent="1-1"/>
+<contactref element="U5" pad="GND"/>
+<contactref element="C3" pad="P$1"/>
+<contactref element="LED4" pad="K"/>
+<wire x1="23.43" y1="45.72" x2="21.59" y2="43.18" width="0" layer="19" extent="1-1"/>
+<wire x1="26.35" y1="56.9795" x2="23.43" y2="45.72" width="0" layer="19" extent="1-1"/>
+<wire x1="-140.97" y1="99.06" x2="26.35" y2="56.9795" width="0" layer="19" extent="1-1"/>
 <wire x1="-33.02" y1="105.41" x2="-140.97" y2="99.06" width="0" layer="19" extent="1-1"/>
 <wire x1="-20.32" y1="60.96" x2="-33.02" y2="105.41" width="0" layer="19" extent="1-1"/>
 <wire x1="-20.32" y1="49.53" x2="-20.32" y2="60.96" width="0" layer="19" extent="1-1"/>
 <wire x1="-20.32" y1="38.1" x2="-20.32" y2="49.53" width="0" layer="19" extent="1-1"/>
-<wire x1="41.59" y1="34.1195" x2="-20.32" y2="38.1" width="0" layer="19" extent="1-1"/>
+<wire x1="11.7" y1="29.21" x2="-20.32" y2="38.1" width="0" layer="19" extent="1-1"/>
+<wire x1="11.7" y1="26.67" x2="11.7" y2="29.21" width="0" layer="19" extent="1-1"/>
+<wire x1="41.59" y1="34.1195" x2="11.7" y2="29.21" width="0" layer="19" extent="1-1"/>
 <wire x1="50.29" y1="38.1" x2="41.59" y2="34.1195" width="0" layer="19" extent="1-1"/>
 <wire x1="50.29" y1="42.28" x2="50.29" y2="38.1" width="0" layer="19" extent="1-1"/>
@@
 <wire x1="35.56" y1="38.1" x2="45.2" y2="40.46" width="0" layer="19" extent="1-1"/>
 </signal>
-<signal name="+5V">
+<signal name="U5V">
 <contactref element="USB1" pad="VBUS1"/>
 <contactref element="USB1" pad="VBUS2"/>
@@
 <wire x1="54.86" y1="42.84" x2="53.86" y2="42.84" width="0" layer="19" extent="1-1"/>
 </signal>
+<signal name="USART_TX">
+<contactref element="U1" pad="P16"/>
+<contactref element="U3" pad="RXD"/>
+<contactref element="ECHO" pad="2"/>
+<wire x1="46.93" y1="47.59" x2="27.94" y2="49.53" width="0" layer="19" extent="1-1"/>
+<wire x1="54.11" y1="51.505" x2="46.93" y2="47.59" width="0" layer="19" extent="1-1"/>
+</signal>
+<signal name="USART_RX">
+<contactref element="U1" pad="P17"/>
+<contactref element="U3" pad="TXD"/>
+<contactref element="ECHO" pad="1"/>
+<wire x1="48.93" y1="49.59" x2="25.4" y2="49.53" width="0" layer="19" extent="1-1"/>
+<wire x1="54.61" y1="51.505" x2="48.93" y2="49.59" width="0" layer="19" extent="1-1"/>
+</signal>
+<signal name="+3V3">
+<contactref element="U3" pad="VCC"/>
+<contactref element="U3" pad="3V3"/>
+<contactref element="C3" pad="P$2"/>
+<wire x1="53.61" y1="51.505" x2="24.83" y2="45.72" width="0" layer="19" extent="1-1"/>
+<wire x1="55.11" y1="51.505" x2="53.61" y2="51.505" width="0" layer="19" extent="1-1"/>
+</signal>
+<signal name="N$33">
+<contactref element="R10" pad="RIGHT"/>
+<contactref element="U3" pad="TNOW"/>
+<wire x1="55.61" y1="51.505" x2="26.4" y2="43.18" width="0" layer="19" extent="1-1"/>
+</signal>
+<signal name="N$34">
+<contactref element="R10" pad="LEFT"/>
+<contactref element="LED4" pad="A"/>
+<wire x1="21.59" y1="44.83" x2="24.4" y2="43.18" width="0" layer="19" extent="1-1"/>
+</signal>
 </signals>

Commit message: 理想ダイオード回路(ディスクリート)の追加
Parts:
- added GND, POW1: (no value), pinhead:1X02
- added POW: 02-JST, con-jst-xh:B2B-XH
- added Q1, Q2, Q3: DMP3056L-7, DMP3056L-7:SOT23
- added R11, R12, R13, R14, R15, R18, R19, R20, R21, R22, R25, R26, R27, R28, R29: 10k, CR0603:CR0603
- added R16, R23, R30: 100k, CR0603:CR0603
- added R17, R24, R31: 0, CR0603:CR0603
- added U6, U7, U8: AP331AWG-7, AP331AWG-7:SOT25
Connections:
- new net N$35: POW1.2, Q1.D, R12.RIGHT
- new net N$37: Q1.G, R11.RIGHT, R16.LEFT, R17.LEFT, R17.RIGHT, U6.OUTPUT
- new net N$38: R12.LEFT, R13.RIGHT, U6.IN-
- new net N$39: R14.LEFT, R15.RIGHT, U6.IN+
- new net N$41: Q2.G, R18.RIGHT, R23.LEFT, R24.LEFT, R24.RIGHT, U7.OUTPUT
- new net N$43: R19.LEFT, R20.RIGHT, U7.IN-
- new net N$44: R21.LEFT, R22.RIGHT, U7.IN+
- new net N$45: POW.2, Q3.D, R26.RIGHT
- new net N$46: Q3.G, R25.RIGHT, R30.LEFT, R31.LEFT, R31.RIGHT, U8.OUTPUT
- new net N$48: R26.LEFT, R27.RIGHT, U8.IN-
- new net N$49: R28.LEFT, R29.RIGHT, U8.IN+
- new net V+: Q1.S, Q2.S, Q3.S, R11.LEFT, R14.RIGHT, R16.RIGHT, R18.LEFT, R21.RIGHT, R23.RIGHT, R25.LEFT, R28.RIGHT, R30.RIGHT, U6.VCC, U7.VCC, U8.VCC
- net GND: now also GND.2
- net GND2: now also GND.1, POW.1, R13.LEFT, R15.LEFT, R20.LEFT, R22.LEFT, R27.LEFT, R29.LEFT, U6.GND, U7.GND, U8.GND
- net U5V: now also Q2.D, R19.RIGHT
- net VCC: now also POW1.1
