File: src/(Eagle)PowerUnit-Bseries(ver1.0).brd (EAGLE design)
At the start: 100 x 100 mm, 161 parts, among them CON1 XT90PW-M, CON2 XT90PW-F, CON3 XT60PW-F, CON4 XT60PW-F, CON5 XT60PW-F, CON6 XT60PW-F, Q2 SSM3J332R, Q4 SSM3J332R, SW1 SS-12SDP2, SW2 RDS-16S-1055-SMT-TR, SW3 SSSS213202, U1 LQFP64, U2 MCP2517FD, U3 CH340E, U5 AP63205WU-7, U7 AP331AWG-7, U9 AP331AWG-7, X1 XRCGB40M000F4M00R0, X2 RH100-24.000-18-1020-EXT-TR, X3 32.768K12.5PI/MC306

Commit message: 電流センサ周りの回路
Parts:
- removed LED2: (no value), led:LED5MM
- removed Q4: SSM3J332R, SSM3J332R:SOT-23F
- removed R1: 100, rcl:0204/7
- added JP6: (no value), pinhead:1X03
- added JP7: (no value), pinhead:1X02
- added RJ45_1, RJ45_2: MTJ-88ARX1-LH, MTJ-88ARX1-LH:MTJ-88ARX1-LH
- added TR1, TR2: 2SC3325, 2SC3325:2SC3325
- added U4, U6, U8: CZ-3A04, CZ3A04:CZ3A07
- C16, C17: value GRM0335C1H120GA01 -> GRM0335C1H6R0BA01D; device GRM0335C1H120GA01:GRM0335C1H120GA01 -> GRM0335C1H6R0BA01D:GRM0335C1H120GA01
- R13: value 2.4Meg -> 150
- R34, R35, R36: value 10k -> 150
- R39: value 100k -> 5.1k
- R40: value 0 -> 5.1k
- U9: value AP331AWG-7 -> CZ-3A04; device AP331AWG-7:SOT25 -> CZ3A04:CZ3A07
- X1: value XRCGB40M000F4M00R0 -> XRCGB40M000F4M01R0; device XRCGB40M000F4M00R0:XRCGB40M000F4M00R0 -> XRCGB40M000F4M01R0:XRCGB40M000F4M00R0
- moved CON6 276.9 mm to (-120.7, 6.35), turned to 0 degrees
- moved CON5 259.3 mm to (-102.9, 6.35), turned to 0 degrees
- moved LED7 258.2 mm to (-134.6, 148.6), turned to 0 degrees
- moved R52 256.5 mm to (-76.2, 156.2), turned to 0 degrees
- moved U$4 255.7 mm to (-132.1, 39.4), turned to 0 degrees
- moved LED6 252.7 mm to (-132.1, 148.6), turned to 0 degrees
- moved R51 251.8 mm to (-72.4, 156.2), turned to 0 degrees
- moved LED5 249.1 mm to (-129.5, 148.6), turned to 0 degrees
- moved C36 246.1 mm to (-76.2, 158.8), turned to 0 degrees
- moved ML1 244.5 mm to (-77.5, 133.3), turned to 0 degrees
- moved CON4 243.1 mm to (-85.1, 6.35), turned to 0 degrees
- moved R50 240.7 mm to (-68.6, 156.2), turned to 0 degrees
- moved P-4 238.9 mm to (-137.2, 61.0), turned to 0 degrees
- moved C1 238.8 mm to (-119.4, 43.2), turned to 0 degrees
- moved R49 234.4 mm to (-64.8, 156.2), turned to 0 degrees
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Connections:
- removed net LED: R1.1
- removed net N$1: CON3.-, EDGE1.P$10, EDGE1.P$11, EDGE1.P$40, EDGE1.P$41, EDGE1.P$42, EDGE1.P$43, EDGE1.P$44, EDGE1.P$6, EDGE1.P$7, EDGE1.P$8, EDGE1.P$9
- removed net N$13: CON6.-, EDGE4.P$10, EDGE4.P$11, EDGE4.P$40, EDGE4.P$41, EDGE4.P$42, EDGE4.P$43, EDGE4.P$44, EDGE4.P$6, EDGE4.P$7, EDGE4.P$8, EDGE4.P$9
- removed net N$18: LED2.A, R1.2
- removed net N$2: CON4.-, EDGE2.P$10, EDGE2.P$11, EDGE2.P$40, EDGE2.P$41, EDGE2.P$42, EDGE2.P$43, EDGE2.P$44, EDGE2.P$6, EDGE2.P$7, EDGE2.P$8, EDGE2.P$9
- removed net N$9: CON5.-, EDGE3.P$10, EDGE3.P$11, EDGE3.P$40, EDGE3.P$41, EDGE3.P$42, EDGE3.P$43, EDGE3.P$44, EDGE3.P$6, EDGE3.P$7, EDGE3.P$8, EDGE3.P$9
- removed net VM2: R35.LEFT, R36.RIGHT, U9.IN-
- new net IN1: EDGE1.P$10, EDGE1.P$11, EDGE1.P$40, EDGE1.P$41, EDGE1.P$42, EDGE1.P$43, EDGE1.P$44, EDGE1.P$6, EDGE1.P$7, EDGE1.P$8, EDGE1.P$9, U4.IN
- new net IN2: EDGE2.P$10, EDGE2.P$11, EDGE2.P$40, EDGE2.P$41, EDGE2.P$42, EDGE2.P$43, EDGE2.P$44, EDGE2.P$6, EDGE2.P$7, EDGE2.P$8, EDGE2.P$9, U6.IN
- new net IN3: EDGE3.P$10, EDGE3.P$11, EDGE3.P$40, EDGE3.P$41, EDGE3.P$42, EDGE3.P$43, EDGE3.P$44, EDGE3.P$6, EDGE3.P$7, EDGE3.P$8, EDGE3.P$9, U8.IN
- new net IN4: EDGE4.P$10, EDGE4.P$11, EDGE4.P$40, EDGE4.P$41, EDGE4.P$42, EDGE4.P$43, EDGE4.P$44, EDGE4.P$6, EDGE4.P$7, EDGE4.P$8, EDGE4.P$9, U9.IN
- new net IP1: CON3.-, U4.IP
- new net IP2: CON4.-, U6.IP
- new net IP3: CON5.-, U8.IP
- new net IP4: CON6.-, U9.IP
- new net N$68: JP7.2, U$1.S
- new net N$69: R35.RIGHT, RJ45_1.LED1_A
- new net N$70: R36.RIGHT, RJ45_2.LED1_A
- new net N$71: RJ45_1.LED1_K, TR1.C
- new net N$72: RJ45_2.LED1_K, TR2.C
- new net N$73: R38.RIGHT, R40.LEFT, TR2.B
- new net N$74: R37.RIGHT, R39.LEFT, TR1.B
- new net N$75: JP6.2, Q2.D, R21.RIGHT
- net +5V: now also R13.RIGHT, R34.RIGHT, R35.LEFT, R36.LEFT, RJ45_1.1, RJ45_1.7, RJ45_2.1, RJ45_2.7; no longer Q4.S, R34.LEFT, R37.RIGHT, R39.RIGHT, U9.VCC
- net CANH: now also RJ45_1.3, RJ45_1.4, RJ45_2.3, RJ45_2.4
- net CANL: now also RJ45_1.5, RJ45_1.6, RJ45_2.5, RJ45_2.6
- net COM_LED: now also R39.RIGHT, R40.RIGHT
- net GND: no longer LED2.K
- net GND2: now also JP7.1, R37.LEFT, RJ45_1.2, RJ45_1.8, RJ45_1.LED2_K, RJ45_2.2, RJ45_2.8, RJ45_2.LED2_K, TR1.E, TR2.E; no longer R36.LEFT, U9.GND
- net N$39: now also X1.1; no longer X1.2
- net N$42: now also X1.2; no longer X1.1
- net N$51: now also RJ45_1.LED2_A; no longer Q4.G, R34.RIGHT, R39.LEFT, R40.LEFT, R40.RIGHT, U9.OUTPUT
- net N$53: now also R34.LEFT, RJ45_2.LED2_A; no longer R13.RIGHT, R37.LEFT, R38.RIGHT, U9.IN+
- net N$55: now also JP6.3; no longer Q2.D, R21.RIGHT
- net U5V: now also JP6.1; no longer Q4.D, R35.RIGHT
Other:
- board size 100 x 100 mm -> 160 x 100 mm

Commit message: OSC周り
Parts:
- added C37, C38, C39, C40, C41, C42, C43: GCM188L81H104KA57, GCM188L81H104K57(0.1uF):GCM188L81H104KA57
- added C44, C45: GRM1885C1H102JA01D, GRM1885C1H102JA01D:GRM18
- added JP8: (no value), pinhead:1X03
- added Q1: SSM3J332R, SSM3J332R:SOT-23F
- added R1: 11.8k, CR0603:CR0603
- added R54: 1.2k, CR0603:CR0603
- added R55: 15.8k, CR0603:CR0603
- added R56: 1.6k, CR0603:CR0603
- added R57: 3.3, CR0603:CR0603
- added R58, R59: 1k, CR0603:CR0603
- added R60, R61: 10k, CR0603:CR0603
- added TP1, TP2: GF063PB103K, GF063P B103K:GF063PB104K
Connections:
- new net CS1_OCD1: C44.L, JP8.3, R58.LEFT, U4.OCD1
- new net CS1_OCD2: C45.L, JP8.1, R59.LEFT, U4.OCD2
- new net CS1_REF1: C41.P$2, R1.LEFT, TP1.CENTER, TP1.LEFT, U4.REF1
- new net CS1_REF2: C42.P$2, R55.LEFT, TP2.CENTER, TP2.LEFT, U4.REF2
- new net CURRENT1: C43.P$2, R57.LEFT
- new net N$1: R57.RIGHT, U4.VOUT
- new net N$13: R54.RIGHT, TP1.RIGHT
- new net N$18: Q1.D, R61.LEFT
- new net N$2: R56.RIGHT, TP2.RIGHT
- new net N$9: JP8.2, Q1.G, R60.LEFT
- net +3V3: now also C37.P$2, R1.RIGHT, R55.RIGHT, R58.RIGHT, R59.RIGHT, R61.RIGHT, U4.VDD
- net GND: no longer C3.P$1
- net GND2: now also C3.P$1, C37.P$1, C41.P$1, C42.P$1, C43.P$1, C44.R, C45.R, Q1.S, R54.LEFT, R56.LEFT, R60.RIGHT, U4.VSS1, U4.VSS2, U6.VSS1, U8.VSS1, U9.VSS1

Commit message: 電源制御系周り
Parts:
- removed IRLB-1, IRLB-2, IRLB-3, IRLB-4: IRLB3813_2, OKUDA_libraries:TO-220AB-PUT
- removed SWITCH: 02-JST, con-jst-xh:B2B-XH
- added C46, C57, C58, C59, C60, C61, C62, C63, C64, C65: GCM188L81H104KA57, GCM188L81H104K57(0.1uF):GCM188L81H104KA57
- added C47, C50, C53, C56: GRM21BC72A105KE01, GRM21BC72A105KE01(1uF):GRM21BC72A105KE01
- added C48, C49, C51, C52, C54, C55: GRM1885C1H102JA01D, GRM1885C1H102JA01D:GRM18
- added INV_SW1, INV_SW2: (no value), pinhead:1X02
- added JP10, JP9: (no value), pinhead:1X03
- added LED2, LED8: SML-E12V8WT86, SML-E12V8WT86:SML-E12V8WT86
- added Q3, Q4, Q5: SSM3J332R, SSM3J332R:SOT-23F
- added Q6, Q7: SQJA16EP-T1_GE3, SQJA16EP-T1_GE3:SQJA16EP-T1_GE3
- added Q8: MTB7D0N06RJ3, MTB7D0N06RJ3:MTB7D0N06RJ3
- added R100, R105, R95: 1.2k, CR0603:CR0603
- added R101, R106, R96: 15.8k, CR0603:CR0603
- added R102, R107, R97: 1.6k, CR0603:CR0603
- added R103, R108, R98: 3.3, CR0603:CR0603
- added R104, R67, R99: 11.8k, CR0603:CR0603
- added R109, R111, R112, R77: 1Meg, CR0603:CR0603
- added R110, R115, R63, R66, R70, R73, R76, R80, R83, R88, R91, R94: 10k, CR0603:CR0603
- added R113, R116: 680, CR0603:CR0603
- added R114: 100, CR0603:CR0603
- added R117: 220, CR0603:CR0603
- added R62, R72, R82, R90: 20k, CR0603:CR0603
- added R64, R68, R69, R71, R74, R78, R79, R81, R84, R86, R87, R89, R92: 1k, CR0603:CR0603
- added R65, R75, R85, R93: 2k, CR0603:CR0603
- added SB1, SB2, SB3, SB4: RSX101VAM-30TR, RSX101VAM-30TR:RSX101VAM-30TR
- added SWITCH_1, SWITCH_2: 02-JST, con-jst-xh:B2B-XH
- added TLP2: TLP152, TLP152:TLP152
- added TP3, TP4, TP5, TP6, TP7, TP8: GF063PB103K, GF063P B103K:GF063PB104K
- added U10, U11, U12, U13: AP331AWG-7, AP331AWG-7:SOT25
- JP1: device pinhead:1X02 -> pinhead:1X03
- LED1, LED3: value (none) -> SML-E12V8WT86; device led:LED5MM -> SML-E12V8WT86:SML-E12V8WT86
- R2, R5: device rcl:0204/7 -> CR0603:CR0603
- R3: value 1kΩ -> 100; device rcl:0204/7 -> CR0603:CR0603
- R4: value 10kΩ -> 10k; device rcl:0204/7 -> CR0603:CR0603
- R6: value 1kΩ -> 1k; device rcl:0204/7 -> CR0603:CR0603
- R61: value 10k -> 1k
- TLP1: value 2227MC-08-03 -> TLP152; device TLP250H:2227MC-08-03 -> TLP152:TLP152
- moved R61 292.0 mm to (-41.9, 168.9)
- moved R60 290.9 mm to (-38.1, 168.9)
- moved R59 278.0 mm to (-34.3, 168.9)
- moved R58 277.2 mm to (-30.5, 168.9)
- moved R57 269.4 mm to (-26.7, 168.9)
- moved C43 266.2 mm to (-67.3, 177.8)
- moved C45 263.1 mm to (-128.3, 171.4)
- moved Q1 256.7 mm to (-147.3, 156.2)
- moved R56 255.0 mm to (-22.9, 168.9)
- moved C44 253.4 mm to (-119.4, 171.4)
- moved C42 252.3 mm to (-64.8, 177.8)
- moved C41 250.6 mm to (-62.2, 177.8)
- moved JP8 246.8 mm to (-121.9, 149.9)
- moved R55 244.5 mm to (-19.1, 168.9)
- moved R54 244.2 mm to (-15.2, 168.9)
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Connections:
- new net CS2_OCD1: C48.L, JP1.3, R68.LEFT, U6.OCD1
- new net CS2_OCD2: C49.L, JP1.1, R69.LEFT, U6.OCD2
- new net CS2_REF1: C39.P$2, R67.LEFT, TP3.CENTER, TP3.LEFT, U6.REF1
- new net CS2_REF2: C40.P$2, R96.LEFT, TP4.CENTER, TP4.LEFT, U6.REF2
- new net CS3_OCD1: C51.L, JP9.3, R78.LEFT, U8.OCD1
- new net CS3_OCD2: C52.L, JP9.1, R79.LEFT, U8.OCD2
- new net CS3_REF1: C58.P$2, R99.LEFT, TP5.CENTER, TP5.LEFT, U8.REF1
- new net CS3_REF2: C59.P$2, R101.LEFT, TP6.CENTER, TP6.LEFT, U8.REF2
- new net CS4_OCD1: C54.L, JP10.3, R86.LEFT, U9.OCD1
- new net CS4_OCD2: C55.L, JP10.1, R87.LEFT, U9.OCD2
- new net CS4_REF1: C62.P$2, R104.LEFT, TP7.CENTER, TP7.LEFT, U9.REF1
- new net CS4_REF2: C63.P$2, R106.LEFT, TP8.CENTER, TP8.LEFT, U9.REF2
- new net CURRENT2: C46.P$2, R98.LEFT, U1.P9
- new net CURRENT3: C60.P$2, R103.LEFT, U1.P10
- new net CURRENT4: C64.P$2, R108.LEFT, U1.P11
- new net N$100: R105.RIGHT, TP7.RIGHT
- new net N$101: R107.RIGHT, TP8.RIGHT
- new net N$102: R108.RIGHT, U9.VOUT
- new net N$103: R12.LEFT, R20.RIGHT, R33.RIGHT, U7.OUTPUT
- new net N$104: C35.P$1, R46.RIGHT, R47.LEFT
- new net N$106: C47.P$1, R64.LEFT, R65.RIGHT, U10.IN-
- new net N$76: R109.RIGHT, R62.LEFT, R63.RIGHT, U10.IN+
- new net N$77: JP1.2, Q3.G, R70.LEFT
- new net N$78: R109.LEFT, R66.RIGHT, SB1.A, U10.OUTPUT
- new net N$79: R95.RIGHT, TP3.RIGHT
- new net N$80: R97.RIGHT, TP4.RIGHT
- new net N$81: R98.RIGHT, U6.VOUT
- new net N$82: R100.RIGHT, TP5.RIGHT
- new net N$83: Q3.D, R71.LEFT, R74.RIGHT
- new net N$84: R72.LEFT, R73.RIGHT, R77.RIGHT, U11.IN+
- new net N$85: R76.RIGHT, R77.LEFT, SB2.A, U11.OUTPUT
- new net N$86: C50.P$1, R74.LEFT, R75.RIGHT, U11.IN-
- new net N$87: JP9.2, Q4.G, R80.LEFT
- new net N$88: Q4.D, R81.LEFT, R84.RIGHT
- new net N$89: R111.RIGHT, R82.LEFT, R83.RIGHT, U12.IN+
- new net N$90: R110.RIGHT, R111.LEFT, SB3.A, U12.OUTPUT
- new net N$91: C53.P$1, R84.LEFT, R85.RIGHT, U12.IN-
- new net N$92: JP10.2, Q5.G, R88.LEFT
- new net N$93: Q5.D, R89.LEFT, R92.RIGHT
- new net N$94: R112.RIGHT, R90.LEFT, R91.RIGHT, U13.IN+
- new net N$95: R112.LEFT, R94.RIGHT, SB4.A, U13.OUTPUT
- new net N$96: C56.P$1, R92.LEFT, R93.RIGHT, U13.IN-
- new net N$98: R102.RIGHT, TP6.RIGHT
- new net N$99: R103.RIGHT, U8.VOUT
- new net SHUTDOWN: R117.RIGHT, SB1.C, SB2.C, SB3.C, SB4.C
- net +3V3: now also C38.P$2, C57.P$2, C61.P$2, R101.RIGHT, R104.RIGHT, R106.RIGHT, R110.LEFT, R62.RIGHT, R66.LEFT, R67.RIGHT, R68.RIGHT, R69.RIGHT, R71.RIGHT, R72.RIGHT, R76.LEFT, R78.RIGHT, R79.RIGHT, R81.RIGHT, R82.RIGHT, R86.RIGHT, R87.RIGHT, R89.RIGHT, R90.RIGHT, R94.LEFT, R96.RIGHT, R99.RIGHT, U10.VCC, U11.VCC, U12.VCC, U13.VCC, U6.VDD, U8.VDD, U9.VDD
- net CURRENT1: now also U1.P8
- net DEBUG_BT: no longer C35.P$1, R46.RIGHT, R47.LEFT
- net GND: now also C65.P$2, INV_SW2.2, Q6.S1, Q6.S2, Q6.S3, Q7.S1, Q7.S2, Q7.S3, R4.LEFT, SWITCH_2.1, TLP1.GND, TLP2.GND; no longer IRLB-1.S, IRLB-2.S, IRLB-3.S, IRLB-4.S, JP1.1, R4.2, TLP1.P$5
- net GND2: now also C38.P$1, C39.P$1, C40.P$1, C46.P$1, C47.P$2, C48.R, C49.R, C50.P$2, C51.R, C52.R, C53.P$2, C54.R, C55.R, C56.P$2, C57.P$1, C58.P$1, C59.P$1, C60.P$1, C61.P$1, C62.P$1, C63.P$1, C64.P$1, Q3.S, Q4.S, Q5.S, R100.LEFT, R102.LEFT, R105.LEFT, R107.LEFT, R63.LEFT, R65.LEFT, R70.RIGHT, R73.LEFT, R75.LEFT, R80.RIGHT, R83.LEFT, R85.LEFT, R88.RIGHT, R91.LEFT, R93.LEFT, R95.LEFT, R97.LEFT, TLP2.CATHODE, U10.GND, U11.GND, U12.GND, U13.GND, U6.VSS2, U8.VSS2, U9.VSS2
- net N$11: now also LED8.K, Q8.D, R6.RIGHT; no longer IRLB-2.P$1, P-3.P$2, P-4.P$2
- net N$12: now also R114.RIGHT, TLP2.VO; no longer IRLB-4.P$1, P-7.P$2, P-8.P$2
- net N$14: now also Q8.G, R114.LEFT, R115.RIGHT; no longer EDGE3.P$28, EDGE3.P$29, EDGE3.P$30, EDGE3.P$31, EDGE3.P$32, EDGE3.P$33, EDGE3.P$34, EDGE3.P$35, EDGE3.P$36, EDGE3.P$37, EDGE3.P$38, EDGE3.P$39, P-5.P$1, P-6.P$1
- net N$15: now also CTRL1.2, CTRL2.2, THRU1.2, TLP1.ANODE; no longer IRLB-3.P$1, P-5.P$2, P-6.P$2
- net N$16: now also R6.LEFT, TLP1.CATHODE; no longer R6.2, TLP1.P$3
- net N$17: now also R2.RIGHT; no longer R2.1
- net N$18: now also R64.RIGHT
- net N$19: now also INV_SW1.2, INV_SW2.1, SWITCH_1.1, SWITCH_2.2; no longer CTRL1.2, CTRL2.2, SWITCH.1, THRU1.2, TLP1.P$2
- net N$20: now also R3.RIGHT, TLP1.VO; no longer R3.1, TLP1.P$6
- net N$21: now also INV_SW1.1, LED3.K, Q8.S, R115.LEFT, SWITCH_1.2; no longer JP1.2, R6.1
- net N$22: now also Q6.G, Q7.G, R3.LEFT, R4.RIGHT; no longer IRLB-1.G, IRLB-2.G, IRLB-3.G, IRLB-4.G, R3.2, R4.1
- net N$24: now also LED3.A, R113.RIGHT; no longer IRLB-2.D, LED3.K
- net N$25: now also R117.LEFT, TLP2.ANODE; no longer EDGE1.P$28, EDGE1.P$29, EDGE1.P$30, EDGE1.P$31, EDGE1.P$32, EDGE1.P$33, EDGE1.P$34, EDGE1.P$35, EDGE1.P$36, EDGE1.P$37, EDGE1.P$38, EDGE1.P$39, P-1.P$1, P-2.P$1
- net N$26: now also EDGE1.P$28, EDGE1.P$29, EDGE1.P$30, EDGE1.P$31, EDGE1.P$32, EDGE1.P$33, EDGE1.P$34, EDGE1.P$35, EDGE1.P$36, EDGE1.P$37, EDGE1.P$38, EDGE1.P$39, LED2.K, Q6.D; no longer P-3.P$1, P-4.P$1
- net N$3: now also LED2.A, R5.RIGHT; no longer LED3.A, R5.1
- net N$43: no longer R12.LEFT, R20.RIGHT, R33.RIGHT, U7.OUTPUT
- net N$7: now also LED8.A, R116.RIGHT; no longer IRLB-1.P$1, P-1.P$2, P-2.P$2
- net N$8: now also EDGE3.P$28, EDGE3.P$29, EDGE3.P$30, EDGE3.P$31, EDGE3.P$32, EDGE3.P$33, EDGE3.P$34, EDGE3.P$35, EDGE3.P$36, EDGE3.P$37, EDGE3.P$38, EDGE3.P$39, Q7.D; no longer P-7.P$1, P-8.P$1
- net VCC: now also C65.P$1, R113.LEFT, R116.LEFT, R2.LEFT, R5.LEFT, TLP1.VCC, TLP2.VCC; no longer R2.2, R5.2, SWITCH.2, TLP1.P$8
Other:
- board size 160 x 100 mm -> 100 x 100 mm

Commit message: ヒューズ選定
Parts:
- removed P-1, P-2, P-3, P-4, P-5, P-6, P-7, P-8: P-SWITCH, OKUDA_libraries:P-SWITCH
- added FUSE1: FUSEHOLDER-3568, FUSEHOLDER-3568:FUSEHOLDER-3568
- added Q9: BSS138, BSS138:SOT-23
- added R118: 220, CR0603:CR0603
- R110: value 10k -> 1Meg
- R111: value 1Meg -> 1k
- R112, R77: value 1Meg -> 10k
- R117: value 220 -> 10k
- R64, R92: value 1k -> 2k
- R66, R76, R88, R94: value 10k -> 1k
- R70, R80: value 10k -> 20k
- R71, R81, R87: value 1k -> 10k
- R72, R82: value 20k -> 2k
- R73, R83: value 10k -> 2k
- R75, R85: value 2k -> 1Meg
- moved C56 318.3 mm to (-40.0, 210.0), turned to 90 degrees
- moved R93 314.0 mm to (-49.0, 213.0), turned to 90 degrees
- moved C55 313.4 mm to (-40.0, 201.0), turned to 90 degrees
- moved R112 312.3 mm to (-46.0, 213.0), turned to 90 degrees
- moved R92 311.8 mm to (-49.0, 209.0), turned to 90 degrees
- moved C54 309.5 mm to (-43.0, 201.0), turned to 90 degrees
- moved R89 308.9 mm to (-53.0, 212.0), turned to 90 degrees
- moved R88 306.6 mm to (-53.0, 208.0), turned to 90 degrees
- moved R94 302.5 mm to (-46.0, 201.0), turned to 90 degrees
- moved R91 300.9 mm to (-49.0, 205.0), turned to 90 degrees
- moved R87 298.9 mm to (-68.0, 213.0), turned to 90 degrees
- moved SB4 298.8 mm to (-57.0, 214.0), turned to 90 degrees
- moved R90 298.6 mm to (-49.0, 201.0), turned to 90 degrees
- moved Q5 296.4 mm to (-53.0, 201.0), turned to 90 degrees
- moved R86 296.3 mm to (-68.0, 209.0), turned to 90 degrees
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Connections:
- removed net N$106: C47.P$1, R64.LEFT, R65.RIGHT, U10.IN-
- removed net N$93: Q5.D, R89.LEFT, R92.RIGHT
- removed net N$94: R112.RIGHT, R90.LEFT, R91.RIGHT, U13.IN+
- removed net N$95: R112.LEFT, R94.RIGHT, SB4.A, U13.OUTPUT
- removed net N$96: C56.P$1, R92.LEFT, R93.RIGHT, U13.IN-
- new net N$105: C47.P$1, R109.RIGHT, R64.LEFT, R65.RIGHT, U10.IN+
- new net N$97: R62.LEFT, R63.RIGHT, U10.IN-
- net +3V3: now also Q1.S, Q3.S, Q4.S, Q5.S, R112.LEFT, R118.RIGHT, R60.LEFT, R70.RIGHT, R74.LEFT, R77.LEFT, R80.RIGHT, R84.LEFT, R87.LEFT, R88.RIGHT; no longer R110.LEFT, R61.RIGHT, R71.RIGHT, R72.RIGHT, R76.LEFT, R81.RIGHT, R82.RIGHT, R86.RIGHT, R87.RIGHT
- net CS1_OCD1: now also C48.L, C51.L, C54.L, JP1.3, JP10.3, JP9.3, R68.LEFT, R78.LEFT, R88.LEFT
- net CS1_OCD2: now also C49.L, C52.L, C55.L, JP1.1, JP10.1, JP9.1, R69.LEFT, R79.LEFT, R89.LEFT
- net CS2_OCD1: no longer C48.L, JP1.3, R68.LEFT
- net CS2_OCD2: no longer C49.L, JP1.1, R69.LEFT
- net CS3_OCD1: no longer C51.L, JP9.3, R78.LEFT
- net CS3_OCD2: no longer C52.L, JP9.1, R79.LEFT
- net CS4_OCD1: no longer C54.L, JP10.3, R86.LEFT
- net CS4_OCD2: no longer C55.L, JP10.1, R87.LEFT
- net GND: now also R111.RIGHT, R61.RIGHT, R63.LEFT, R71.LEFT, R76.RIGHT, R81.LEFT, R86.RIGHT, R91.LEFT
- net GND2: now also Q1.D, Q3.D, Q4.D, Q5.D, Q9.S, R111.LEFT, R117.LEFT, R61.LEFT, R64.RIGHT, R72.RIGHT, R76.LEFT, R82.RIGHT, R86.LEFT, R92.RIGHT; no longer Q1.S, Q3.S, Q4.S, Q5.S, R60.RIGHT, R63.LEFT, R70.RIGHT, R75.LEFT, R80.RIGHT, R85.LEFT, R88.RIGHT, R91.LEFT
- net N$18: now also JP1.2, Q3.G, R77.RIGHT; no longer Q1.D, R61.LEFT, R64.RIGHT
- net N$25: now also CON1.+, FUSE1.R1, FUSE1.R2; no longer R117.LEFT, TLP2.ANODE
- net N$76: now also R74.RIGHT, R75.LEFT, SB2.A, U11.OUTPUT; no longer R109.RIGHT, R62.LEFT, R63.RIGHT, U10.IN+
- net N$77: now also R71.RIGHT, U11.IN-; no longer JP1.2, Q3.G
- net N$83: now also C50.P$1, R72.LEFT, R73.RIGHT, R75.RIGHT, U11.IN+; no longer Q3.D, R71.LEFT, R74.RIGHT
- net N$84: now also JP9.2, Q4.G, R87.RIGHT; no longer R72.LEFT, R73.RIGHT, R77.RIGHT, U11.IN+
- net N$85: now also R84.RIGHT, R85.LEFT, SB3.A, U12.OUTPUT; no longer R76.RIGHT, R77.LEFT, SB2.A, U11.OUTPUT
- net N$86: now also R80.LEFT, R81.RIGHT, U12.IN-; no longer C50.P$1, R74.LEFT, R75.RIGHT, U11.IN-
- net N$87: now also C53.P$1, R82.LEFT, R83.RIGHT, R85.RIGHT, U12.IN+; no longer JP9.2, Q4.G, R80.LEFT
- net N$88: now also JP10.2, Q5.G, R112.RIGHT; no longer Q4.D, R81.LEFT, R84.RIGHT
- net N$89: now also R110.LEFT, R94.RIGHT, SB4.A, U13.OUTPUT; no longer R111.RIGHT, R82.LEFT, R83.RIGHT, U12.IN+
- net N$9: now also R60.RIGHT; no longer R60.LEFT
- net N$90: now also R90.LEFT, R91.RIGHT, U13.IN-; no longer R110.RIGHT, R111.LEFT, SB3.A, U12.OUTPUT
- net N$91: now also C56.P$1, R110.RIGHT, R92.LEFT, R93.RIGHT, U13.IN+; no longer C53.P$1, R84.LEFT, R85.RIGHT, U12.IN-
- net N$92: now also Q9.D, R118.LEFT, TLP2.ANODE; no longer JP10.2, Q5.G, R88.LEFT
- net SHUTDOWN: now also Q9.G
- net VCC: now also FUSE1.L1, FUSE1.L2; no longer CON1.+

Commit message: kairozunoseiri
Parts:
- removed TLP2: TLP152, TLP152:TLP152
- added C66, C67, C68, C71: GRM21BC72A105KE01, GRM21BC72A105KE01(1uF):GRM21BC72A105KE01
- added C70: GCM188L81H104KA57, GCM188L81H104K57(0.1uF):GCM188L81H104KA57
- added Q10: SQJA16EP-T1_GE3, SQJA16EP-T1_GE3:SQJA16EP-T1_GE3
- added R119, R121: 10k, CR0603:CR0603
- added R120: 1.8k, CR0603:CR0603
- added R122: 300, CR0603:CR0603
- added R123: 270, CR0603:CR0603
- added R124, R125: 10, CR0603:CR0603
- added THRU2: 02-JST, con-jst-xh:B2B-XH
- added TLP3: TLP152, TLP152:TLP152
- added U14, U15: TCK420G, TCK420G:TCK420G
- added U16, U19: TC7SH00FULJ, TC7SH00FULJ:SSOP5-P-0.65A
- added U17, U18, U21, U22: TC7S14F, TC7S14F:TC7S14F
- added U20: TLP293, TLP293_Mylib:TLP293
- added ZD1: MMSZ5231B-TP, MMSZ5231B-TP:MMSZ5231B-TP
- added ZD2, ZD3, ZD4, ZD5: MMBZ5248B-TP, MMBZ5248B-TP:MMBZ5248B-TP
- C1: value 50ZLH1000MEFC16X25 -> 50MXG3300MEFCSN22X30; device 50ZLH1000MEFC16X25(1000uF):50ZLH1000MEFC16X25 -> 50MXG3300MEFCSN22X30:50MXG3300MEFCSN22X30
- C2: value GCM188L81H104KA57 -> GRM21BC72A105KE01; device GCM188L81H104K57(0.1uF):GCM188L81H104KA57 -> GRM21BC72A105KE01(1uF):GRM21BC72A105KE01
- R114: value 100 -> 820
- R3: value 100 -> 1
- R4: value 10k -> 220
- R6: value 1k -> 820
- moved R6 262.6 mm to (-226.0, -72.0)
- moved R4 258.0 mm to (-220.0, -66.0)
- moved R3 251.7 mm to (-214.0, -60.0)
- moved C2 233.3 mm to (-205.0, -48.0)
- moved C1 62.7 mm to (13.0, 13.0)
Connections:
- net VM1 renamed N$113
- new net 5V1: R121.RIGHT, R123.LEFT, U16.VCC, U17.VCC, U18.VCC, U19.VCC, U21.VCC, ZD1.CATHODE
- new net DISABLE: U1.P20, U22.IN
- new net EMERGENCY: R120.RIGHT, U14.VCT, U15.VCT, U18.IN, U21.OUT
- new net N$106: R122.LEFT, U19.OUT
- new net N$107: U16.INA, U18.OUT
- new net N$108: U16.OUT, U19.INA, U19.INB
- new net N$109: R121.LEFT, U20.COLLECTOR, U21.IN
- new net N$110: R122.RIGHT, TLP3.ANODE
- new net N$111: C66.P$1, C68.P$1, EDGE1.P$12, EDGE1.P$13, EDGE1.P$14, EDGE1.P$15, EDGE1.P$16, EDGE1.P$17, EDGE1.P$18, EDGE1.P$19, EDGE1.P$20, EDGE1.P$21, EDGE1.P$22, EDGE1.P$23, EDGE2.P$12, EDGE2.P$13, EDGE2.P$14, EDGE2.P$15, EDGE2.P$16, EDGE2.P$17, EDGE2.P$18, EDGE2.P$19, EDGE2.P$20, EDGE2.P$21, EDGE2.P$22, EDGE2.P$23, EDGE3.P$12, EDGE3.P$13, EDGE3.P$14, EDGE3.P$15, EDGE3.P$16, EDGE3.P$17, EDGE3.P$18, EDGE3.P$19, EDGE3.P$20, EDGE3.P$21, EDGE3.P$22, EDGE3.P$23, EDGE4.P$12, EDGE4.P$13, EDGE4.P$14, EDGE4.P$15, EDGE4.P$16, EDGE4.P$17, EDGE4.P$18, EDGE4.P$19, EDGE4.P$20, EDGE4.P$21, EDGE4.P$22, EDGE4.P$23, Q6.S1, Q6.S2, Q6.S3, Q7.S1, Q7.S2, Q7.S3, R3.LEFT, R5.LEFT, U14.VOUT, U15.VOUT, ZD2.ANODE, ZD4.ANODE
- new net N$112: Q6.G, R124.LEFT, ZD2.CATHODE
- new net N$93: C71.P$1, R120.LEFT, U17.IN
- new net N$94: R4.RIGHT, U20.ANODE
- new net N$95: R6.LEFT, TLP3.VO
- new net N$96: Q10.G, R119.RIGHT, R6.RIGHT, ZD5.CATHODE
- net +3V3: now also U22.VCC
- net GND: now also C1.CATHODE, C66.P$2, C67.P$2, C68.P$2, C70.P$2, C71.P$2, EDGE1.P$28, EDGE1.P$29, EDGE1.P$30, EDGE1.P$31, EDGE1.P$32, EDGE1.P$33, EDGE1.P$34, EDGE1.P$35, EDGE1.P$36, EDGE1.P$37, EDGE1.P$38, EDGE1.P$39, EDGE2.P$28, EDGE2.P$29, EDGE2.P$30, EDGE2.P$31, EDGE2.P$32, EDGE2.P$33, EDGE2.P$34, EDGE2.P$35, EDGE2.P$36, EDGE2.P$37, EDGE2.P$38, EDGE2.P$39, EDGE3.P$28, EDGE3.P$29, EDGE3.P$30, EDGE3.P$31, EDGE3.P$32, EDGE3.P$33, EDGE3.P$34, EDGE3.P$35, EDGE3.P$36, EDGE3.P$37, EDGE3.P$38, EDGE3.P$39, EDGE4.P$28, EDGE4.P$29, EDGE4.P$30, EDGE4.P$31, EDGE4.P$32, EDGE4.P$33, EDGE4.P$34, EDGE4.P$35, EDGE4.P$36, EDGE4.P$37, EDGE4.P$38, EDGE4.P$39, LED2.K, Q10.S1, Q10.S2, Q10.S3, R119.LEFT, TLP3.CATHODE, TLP3.GND, U14.GND, U15.GND, U16.GND, U17.GND, U18.GND, U19.GND, U20.EMITTER, U21.GND, ZD1.ANODE, ZD3.ANODE, ZD5.ANODE; no longer C1.C, Q6.S1, Q6.S2, Q6.S3, Q7.S1, Q7.S2, Q7.S3, R4.LEFT, TLP2.GND
- net GND2: now also TLP1.CATHODE, U22.GND; no longer TLP2.CATHODE
- net N$11: now also Q10.D, R3.RIGHT; no longer LED8.K, Q8.D, R6.RIGHT
- net N$12: now also TLP1.VO; no longer TLP2.VO
- net N$14: now also ZD3.CATHODE
- net N$15: now also R4.LEFT, THRU2.2; no longer TLP1.ANODE
- net N$16: now also LED8.K, Q8.D, U20.CATHODE; no longer R6.LEFT, TLP1.CATHODE
- net N$20: now also Q7.G, R125.LEFT, ZD4.CATHODE; no longer R3.RIGHT, TLP1.VO
- net N$21: now also THRU2.1
- net N$22: now also U16.INB, U17.OUT; no longer Q6.G, Q7.G, R3.LEFT, R4.RIGHT
- net N$26: now also R124.RIGHT, U14.VGATE2; no longer EDGE1.P$28, EDGE1.P$29, EDGE1.P$30, EDGE1.P$31, EDGE1.P$32, EDGE1.P$33, EDGE1.P$34, EDGE1.P$35, EDGE1.P$36, EDGE1.P$37, EDGE1.P$38, EDGE1.P$39, EDGE2.P$28, EDGE2.P$29, EDGE2.P$30, EDGE2.P$31, EDGE2.P$32, EDGE2.P$33, EDGE2.P$34, EDGE2.P$35, EDGE2.P$36, EDGE2.P$37, EDGE2.P$38, EDGE2.P$39, LED2.K, Q6.D
- net N$8: now also R125.RIGHT, U15.VGATE2; no longer EDGE3.P$28, EDGE3.P$29, EDGE3.P$30, EDGE3.P$31, EDGE3.P$32, EDGE3.P$33, EDGE3.P$34, EDGE3.P$35, EDGE3.P$36, EDGE3.P$37, EDGE3.P$38, EDGE3.P$39, EDGE4.P$28, EDGE4.P$29, EDGE4.P$30, EDGE4.P$31, EDGE4.P$32, EDGE4.P$33, EDGE4.P$34, EDGE4.P$35, EDGE4.P$36, EDGE4.P$37, EDGE4.P$38, EDGE4.P$39, Q7.D
- net N$92: now also TLP1.ANODE; no longer TLP2.ANODE
- net SHUTDOWN: now also U22.OUT
- net VCC: now also C1.ANODE, C67.P$1, C70.P$1, Q6.D, Q7.D, R123.RIGHT, TLP3.VCC, U14.VIN, U15.VIN; no longer C1.A, EDGE1.P$12, EDGE1.P$13, EDGE1.P$14, EDGE1.P$15, EDGE1.P$16, EDGE1.P$17, EDGE1.P$18, EDGE1.P$19, EDGE1.P$20, EDGE1.P$21, EDGE1.P$22, EDGE1.P$23, EDGE2.P$12, EDGE2.P$13, EDGE2.P$14, EDGE2.P$15, EDGE2.P$16, EDGE2.P$17, EDGE2.P$18, EDGE2.P$19, EDGE2.P$20, EDGE2.P$21, EDGE2.P$22, EDGE2.P$23, EDGE3.P$12, EDGE3.P$13, EDGE3.P$14, EDGE3.P$15, EDGE3.P$16, EDGE3.P$17, EDGE3.P$18, EDGE3.P$19, EDGE3.P$20, EDGE3.P$21, EDGE3.P$22, EDGE3.P$23, EDGE4.P$12, EDGE4.P$13, EDGE4.P$14, EDGE4.P$15, EDGE4.P$16, EDGE4.P$17, EDGE4.P$18, EDGE4.P$19, EDGE4.P$20, EDGE4.P$21, EDGE4.P$22, EDGE4.P$23, R5.LEFT, TLP2.VCC
