File: src/(Eagle)PowerUnit-Bseries(ver1.0).brd (EAGLE design)
At the start: 100 x 100 mm, 312 parts, among them CON1 XT90PW-M, CON2 XT90PW-F, CON3 XT60PW-F, CON4 XT60PW-F, CON5 XT60PW-F, CON6 XT60PW-F, Q1 SSM3J332R, Q10 SQJA16EP-T1_GE3, Q2 SSM3J332R, Q3 SSM3J332R, Q4 SSM3J332R, Q5 SSM3J332R, Q6 SQJA16EP-T1_GE3, Q7 SQJA16EP-T1_GE3, Q8 MTB7D0N06RJ3, Q9 BSS138, SW1 SS-12SDP2, SW2 RDS-16S-1055-SMT-TR, SW3 SSSS213202, U1 LQFP64, U10 AP331AWG-7, U11 AP331AWG-7, U12 AP331AWG-7, U13 AP331AWG-7, U14 TCK420G, U15 TCK420G, U16 TC7SH00FULJ, U17 TC7S14F, U18 TC7S14F, U19 TC7SH00FULJ, U2 MCP2517FD, U20 TLP293, U21 TC7S14F, U22 TC7S14F, U3 CH340E, U4 CZ-3A04, U5 AP63205WU-7, U6 CZ-3A04, U7 AP331AWG-7, U8 CZ-3A04, U9 CZ-3A04, X1 XRCGB40M000F4M01R0, X2 RH100-24.000-18-1020-EXT-TR, X3 32.768K12.5PI/MC306

Commit message: DGND未選別のところまで
Parts:
- removed Q3, Q4, Q5: SSM3J332R, SSM3J332R:SOT-23F
- removed Q7: SQJA16EP-T1_GE3, SQJA16EP-T1_GE3:SQJA16EP-T1_GE3
- removed Q8: MTB7D0N06RJ3, MTB7D0N06RJ3:MTB7D0N06RJ3
- removed Q9: BSS138, BSS138:SOT-23
- removed R109, R110, R85: 1Meg, CR0603:CR0603
- removed R111, R79, R84, R86, R88, R89, R94: 1k, CR0603:CR0603
- removed R112, R117, R81, R87, R91: 10k, CR0603:CR0603
- removed R114: 820, CR0603:CR0603
- removed R118: 220, CR0603:CR0603
- removed R125: 10, CR0603:CR0603
- removed R80, R90: 20k, CR0603:CR0603
- removed R82, R83, R92, R93: 2k, CR0603:CR0603
- removed SWITCH_1, SWITCH_2: 02-JST, con-jst-xh:B2B-XH
- removed ZD3, ZD4: MMBZ5248B-TP, MMBZ5248B-TP:MMBZ5248B-TP
- added C69: GRM21BC72A105KE01, GRM21BC72A105KE01(1uF):GRM21BC72A105KE01
- added D3: PJSD12TS, PJSD12TS:SOD-523
- added Q11, Q12: TMBT3906, TMBT3906:TMBT3906
- added SB5: V2P22LHM3/H, V2P22LHM3:V2P22LHM3/H
- added SB6: 1SS404,H3F, 1SS404,H3F:1SS404,H3F
- added SB7: RSX101VAM-30TR, RSX101VAM-30TR:RSX101VAM-30TR
- added SW4, SW5: 2MS1-T2-B4-M2-Q-E-S, 2MS1-T2-B4-M2-Q-E-S:2MS1-T2-B4-M2-Q-E-S
- added TR3: 2SC3325, 2SC3325:2SC3325
- added U23, U25: TC7S14F, TC7S14F:TC7S14F
- added U24: MCP6541T-I/LT, MCP6541T-I:SC-70-5
- added U26: TC7SH00FULJ, TC7SH00FULJ:SSOP5-P-0.65A
- C1: value 50MXG3300MEFCSN22X30 -> 50SEV470M16X16.5; device 50MXG3300MEFCSN22X30:50MXG3300MEFCSN22X30 -> 50SEV470M16X16.5:50SEV470M16X16.5
- C68: value GRM21BC72A105KE01 -> GRM0335C1H620GA01D; device GRM21BC72A105KE01(1uF):GRM21BC72A105KE01 -> GRM0335C1H620GA01D:GRM0335C1E240GA01D
- Q1: value SSM3J332R -> SQJA16EP-T1_GE3; device SSM3J332R:SOT-23F -> SQJA16EP-T1_GE3:SQJA16EP-T1_GE3
- R12: value 2.4Meg -> 10k
- R120: value 1.8k -> 620
- R22: value 10k -> 20k
- R23, R24, R63, R77: value 10k -> 1k
- R32: value 100k -> 10k
- R33: value 0 -> 1k
- R61, R66: value 1k -> 20k
- R62, R70: value 20k -> 1k
- R64, R73: value 2k -> 1k
- R65: value 2k -> 10k
- R72: value 2k -> 20k
- R74: value 1k -> 0
- R75: value 1Meg -> ∞
- R76: value 1k -> 36k
- R78: value 1k -> 100
- U10, U13: value AP331AWG-7 -> TC7S14F; device AP331AWG-7:SOT25 -> TC7S14F:TC7S14F
- U11, U12, U7: value AP331AWG-7 -> MCP6541T-I/LT; device AP331AWG-7:SOT25 -> MCP6541T-I:SC-70-5
- U15: value TCK420G -> TCKE805NAWSON10B_TOS-REC; device TCK420G:TCK420G -> TCKE805NA:WSON10B_TOS-RIC
- moved R78 396.4 mm to (-272.0, -136.0), turned to 0 degrees
- moved R77 383.3 mm to (-261.0, -130.0), turned to 0 degrees
- moved R76 360.3 mm to (-239.0, -119.0), turned to 0 degrees
- moved R75 353.9 mm to (-239.0, -116.0), turned to 0 degrees
- moved R74 347.6 mm to (-239.0, -113.0), turned to 0 degrees
- moved R122 271.3 mm to (-165.0, 162.0)
- moved R123 271.3 mm to (-167.0, 159.0)
- moved R124 271.3 mm to (-167.0, 123.0)
- moved ZD1 271.3 mm to (-166.0, 155.0)
- moved ZD2 271.3 mm to (-167.0, 146.0)
- moved ZD5 271.3 mm to (-167.0, 132.0)
- moved U22 268.0 mm to (-179.0, 120.0)
- moved C56 220.6 mm to (-173.0, 34.0), turned to 0 degrees
- moved C55 219.2 mm to (-182.0, 34.0), turned to 0 degrees
- moved C54 212.4 mm to (-178.0, 37.0), turned to 0 degrees
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Connections:
- new net N$114: JP10.2, U25.IN
- new net N$115: R73.RIGHT, U25.OUT
- new net N$116: R76.RIGHT, U15.ILIM
- new net N$117: C68.1, U15.DVDT
- new net N$118: R78.RIGHT, TLP1.ANODE
- new net N$119: SB7.A, U22.OUT
- net +3V3: now also R21.LEFT, R24.RIGHT, R33.RIGHT, R63.RIGHT, R64.RIGHT, R65.LEFT, R71.LEFT, U11.VDD, U12.VDD, U23.VCC, U24.VDD, U25.VCC, U26.VCC, U7.VDD; no longer Q1.S, Q3.S, Q4.S, Q5.S, R112.LEFT, R118.RIGHT, R62.RIGHT, R66.LEFT, R68.RIGHT, R74.LEFT, R77.LEFT, R78.RIGHT, R79.RIGHT, R80.RIGHT, R84.LEFT, R87.LEFT, R88.RIGHT, R89.RIGHT, R90.RIGHT, R94.LEFT, U11.VCC, U12.VCC
- net +5V: now also Q11.E; no longer R20.LEFT, R23.RIGHT, U7.VCC
- net CS1_OCD1: now also R24.LEFT, R63.LEFT, R69.LEFT; no longer R68.LEFT, R78.LEFT, R88.LEFT
- net CS1_OCD2: now also R33.LEFT, R64.LEFT, R70.LEFT; no longer R69.LEFT, R79.LEFT, R89.LEFT
- net EMERGENCY: no longer U15.VCT
- net GND: now also SW5.O; no longer C67.P$2, C68.P$2, R111.RIGHT, R61.RIGHT, R63.LEFT, R71.LEFT, R76.RIGHT, R81.LEFT, R86.RIGHT, R91.LEFT, SWITCH_2.1, U15.GND, ZD3.ANODE
- net GND2: now also C67.P$2, C68.2, C69.P$2, D3.A, R12.LEFT, R20.LEFT, R22.RIGHT, R61.RIGHT, R66.RIGHT, R75.LEFT, SB6.A, U11.VSS, U12.VSS, U15.GND1, U15.GND2, U15.GND3, U15.GND4, U15.GND5, U23.GND, U24.VSS, U25.GND, U26.GND, U7.VSS; no longer Q1.D, Q3.D, Q4.D, Q5.D, Q9.S, R111.LEFT, R117.LEFT, R22.LEFT, R24.LEFT, R61.LEFT, R64.RIGHT, R65.LEFT, R73.LEFT, R82.RIGHT, R83.LEFT, R86.LEFT, R92.RIGHT, R93.LEFT, U11.GND, U12.GND, U7.GND
- net N$103: now also Q11.C, Q2.G, R32.LEFT; no longer R12.LEFT, R33.RIGHT, U7.OUTPUT
- net N$105: now also R23.RIGHT, U10.OUT; no longer C47.P$1, R109.RIGHT, R64.LEFT, R65.RIGHT, U10.IN+
- net N$111: now also Q1.S1, Q1.S2, Q1.S3, SB5.A; no longer C68.P$1, Q7.S1, Q7.S2, Q7.S3, U15.VOUT, ZD4.ANODE
- net N$112: now also Q1.G
- net N$113: now also R62.RIGHT, U23.OUT; no longer R21.LEFT, R22.RIGHT, U7.IN-
- net N$12: now also R77.LEFT; no longer R114.RIGHT
- net N$14: now also R77.RIGHT, TR3.B; no longer Q8.G, R114.LEFT, ZD3.CATHODE
- net N$16: now also TR3.C; no longer Q8.D
- net N$18: now also R60.RIGHT, R61.LEFT, U11.IN-; no longer JP1.2, Q3.G, R77.RIGHT
- net N$19: now also SW4.O, SW5.P; no longer SWITCH_1.1, SWITCH_2.2
- net N$20: now also C67.P$1, D3.C, JP6.2, R74.RIGHT, U15.VIN1, U15.VIN2, U15.VIN3; no longer Q7.G, R125.LEFT, ZD4.CATHODE
- net N$21: now also SW4.P, TR3.E; no longer Q8.S, SWITCH_1.2
- net N$43: now also R21.RIGHT, R22.LEFT, U7.IN-; no longer Q2.G, R32.LEFT, R33.LEFT
- net N$47: now also Q11.B, Q12.B, Q12.C; no longer R23.LEFT, R24.RIGHT, U7.IN+
- net N$75: now also C69.P$1, Q12.E, SB6.C, U15.VOUT1, U15.VOUT2, U15.VOUT3; no longer JP6.2, R21.RIGHT
- net N$76: now also C50.P$1, R62.LEFT, U11.IN+; no longer R74.RIGHT, R75.LEFT, SB2.A, U11.OUTPUT
- net N$77: now also SB2.A, U11.OUT; no longer R70.LEFT, R71.RIGHT, U11.IN-
- net N$78: now also C47.P$1, R23.LEFT, U7.IN+; no longer R109.LEFT, R66.RIGHT, SB1.A, U10.OUTPUT
- net N$8: now also R74.LEFT, R75.RIGHT, U15.EN/UVLO; no longer R125.RIGHT, U15.VGATE2
- net N$83: now also JP1.2, U23.IN; no longer C50.P$1, R72.LEFT, R73.RIGHT, R75.RIGHT, U11.IN+
- net N$84: now also R65.RIGHT, R66.LEFT, U12.IN-; no longer JP9.2, Q4.G, R87.RIGHT
- net N$85: now also C53.P$1, R68.LEFT, U12.IN+; no longer R84.RIGHT, R85.LEFT, SB3.A, U12.OUTPUT
- net N$86: now also SB3.A, U12.OUT; no longer R80.LEFT, R81.RIGHT, U12.IN-
- net N$87: now also JP9.2, U13.IN; no longer C53.P$1, R82.LEFT, R83.RIGHT, R85.RIGHT, U12.IN+
- net N$88: now also R68.RIGHT, U13.OUT; no longer JP10.2, Q5.G, R112.RIGHT
- net N$89: now also R71.RIGHT, R72.LEFT, U24.IN-; no longer R110.LEFT, R94.RIGHT, SB4.A, U13.OUTPUT
- net N$9: now also U10.IN; no longer Q1.G, R60.RIGHT
- net N$90: now also C56.P$1, R73.LEFT, U24.IN+; no longer R90.LEFT, R91.RIGHT, U13.IN-
- net N$91: now also SB4.A, U24.OUT; no longer C56.P$1, R110.RIGHT, R92.LEFT, R93.RIGHT, U13.IN+
- net N$92: now also R78.LEFT, U26.OUT; no longer Q9.D, R118.LEFT, TLP1.ANODE
- net N$97: now also SB1.A, U7.OUT; no longer R62.LEFT, R63.RIGHT, U10.IN-
- net SHUTDOWN: now also SB7.C, U26.INA, U26.INB; no longer Q9.G, R117.RIGHT, U22.OUT
- net VCC: now also Q1.D, SB5.C; no longer C67.P$1, Q7.D, U15.VIN
