File: src/(Eagle)PowerUnit-Bseries(ver1.0).sch (EAGLE design)
At the start: 161 parts, among them CON1 XT90PW-M, CON2 XT90PW-F, CON3 XT60PW-F, CON4 XT60PW-F, CON5 XT60PW-F, CON6 XT60PW-F, Q2 SSM3J332R, Q4 SSM3J332R, SW1 SS-12SDP2, SW2 RDS-16S-1055-SMT-TR, SW3 SSSS213202, U1 LQFP64, U2 MCP2517FD, U3 CH340E, U5 AP63205WU-7, U7 AP331AWG-7, U9 AP331AWG-7, X1 XRCGB40M000F4M00R0, X2 RH100-24.000-18-1020-EXT-TR, X3 32.768K12.5PI/MC306

Commit message: 電流センサ周りの回路
Parts:
- removed LED2: (no value), led:LED5MM
- removed Q4: SSM3J332R, SSM3J332R:SSM3J332R
- removed R1: 100, rcl:R-EU_0204/7
- added JP6: (no value), pinhead:PINHD-1X3
- added JP7: (no value), pinhead:PINHD-1X2
- added RJ45_1, RJ45_2: MTJ-88ARX1-LH, MTJ-88ARX1-LH:MTJ-88ARX1-LH
- added TR1, TR2: 2SC3325, 2SC3325:2SC3325
- added U4, U6, U8: CZ-3A04, CZ3A04:CZ-3A04
- C16, C17: value GRM0335C1H120GA01 -> GRM0335C1H6R0BA01D; device GRM0335C1H120GA01:GRM0335C1H120GA01 -> GRM0335C1H6R0BA01D:GRM0335C1H6R0BA01D
- R13: value 2.4Meg -> 150
- R34, R35, R36: value 10k -> 150
- R39: value 100k -> 5.1k
- R40: value 0 -> 5.1k
- U9: value AP331AWG-7 -> CZ-3A04; device AP331AWG-7:AP331AWG-7 -> CZ3A04:CZ-3A04
- X1: value XRCGB40M000F4M00R0 -> XRCGB40M000F4M01R0; device XRCGB40M000F4M00R0:XRCGB40M000F4M00R0 -> XRCGB40M000F4M01R0:XRCGB40M000F4M01R0
Connections:
- removed net LED: R1.1
- removed net N$1: CON3.-, EDGE1.P10, EDGE1.P11, EDGE1.P40, EDGE1.P41, EDGE1.P42, EDGE1.P43, EDGE1.P44, EDGE1.P6, EDGE1.P7, EDGE1.P8, EDGE1.P9
- removed net N$13: CON6.-, EDGE4.P10, EDGE4.P11, EDGE4.P40, EDGE4.P41, EDGE4.P42, EDGE4.P43, EDGE4.P44, EDGE4.P6, EDGE4.P7, EDGE4.P8, EDGE4.P9
- removed net N$18: LED2.A, R1.2
- removed net N$2: CON4.-, EDGE2.P10, EDGE2.P11, EDGE2.P40, EDGE2.P41, EDGE2.P42, EDGE2.P43, EDGE2.P44, EDGE2.P6, EDGE2.P7, EDGE2.P8, EDGE2.P9
- removed net N$9: CON5.-, EDGE3.P10, EDGE3.P11, EDGE3.P40, EDGE3.P41, EDGE3.P42, EDGE3.P43, EDGE3.P44, EDGE3.P6, EDGE3.P7, EDGE3.P8, EDGE3.P9
- removed net VM2: R35.LEFT, R36.RIGHT, U9.IN-
- new net IN1: EDGE1.P10, EDGE1.P11, EDGE1.P40, EDGE1.P41, EDGE1.P42, EDGE1.P43, EDGE1.P44, EDGE1.P6, EDGE1.P7, EDGE1.P8, EDGE1.P9, U4.IN
- new net IN2: EDGE2.P10, EDGE2.P11, EDGE2.P40, EDGE2.P41, EDGE2.P42, EDGE2.P43, EDGE2.P44, EDGE2.P6, EDGE2.P7, EDGE2.P8, EDGE2.P9, U6.IN
- new net IN3: EDGE3.P10, EDGE3.P11, EDGE3.P40, EDGE3.P41, EDGE3.P42, EDGE3.P43, EDGE3.P44, EDGE3.P6, EDGE3.P7, EDGE3.P8, EDGE3.P9, U8.IN
- new net IN4: EDGE4.P10, EDGE4.P11, EDGE4.P40, EDGE4.P41, EDGE4.P42, EDGE4.P43, EDGE4.P44, EDGE4.P6, EDGE4.P7, EDGE4.P8, EDGE4.P9, U9.IN
- new net IP1: CON3.-, U4.IP
- new net IP2: CON4.-, U6.IP
- new net IP3: CON5.-, U8.IP
- new net IP4: CON6.-, U9.IP
- new net N$68: JP7.2, U$1.S
- new net N$69: R35.RIGHT, RJ45_1.LED1_A
- new net N$70: R36.RIGHT, RJ45_2.LED1_A
- new net N$71: RJ45_1.LED1_K, TR1.C
- new net N$72: RJ45_2.LED1_K, TR2.C
- new net N$73: R38.RIGHT, R40.LEFT, TR2.B
- new net N$74: R37.RIGHT, R39.LEFT, TR1.B
- new net N$75: JP6.2, Q2.DRAIN, R21.RIGHT
- net +5V: now also R13.RIGHT, R34.RIGHT, R35.LEFT, R36.LEFT, RJ45_1.1, RJ45_1.7, RJ45_2.1, RJ45_2.7; no longer Q4.SOURCE, R34.LEFT, R37.RIGHT, R39.RIGHT, U9.VCC
- net CANH: now also RJ45_1.3, RJ45_1.4, RJ45_2.3, RJ45_2.4
- net CANL: now also RJ45_1.5, RJ45_1.6, RJ45_2.5, RJ45_2.6
- net COM_LED: now also R39.RIGHT, R40.RIGHT
- net GND: no longer LED2.C
- net GND2: now also JP7.1, R37.LEFT, RJ45_1.2, RJ45_1.8, RJ45_1.LED2_K, RJ45_2.2, RJ45_2.8, RJ45_2.LED2_K, TR1.E, TR2.E; no longer R36.LEFT, U9.GND
- net N$39: now also X1.1; no longer X1.2
- net N$42: now also X1.2; no longer X1.1
- net N$51: now also RJ45_1.LED2_A; no longer Q4.GATE, R34.RIGHT, R39.LEFT, R40.LEFT, R40.RIGHT, U9.OUTPUT
- net N$53: now also R34.LEFT, RJ45_2.LED2_A; no longer R13.RIGHT, R37.LEFT, R38.RIGHT, U9.IN+
- net N$55: now also JP6.3; no longer Q2.DRAIN, R21.RIGHT
- net U5V: now also JP6.1; no longer Q4.DRAIN, R35.RIGHT
Other:
- note added: "BOOT0=0 - Boot from main flash memory"
- note added: "BOOT0=1 - Boot from system memory(boot loader)"
- note removed: "BOOTモード->BOOT0=1,BOOT1=0"
- note removed: "MDC LED check"
- moved on the sheet: C1, C10, C11, C12, C13, C14, C15, C16, C17, C2, C3, C4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

Commit message: OSC周り
Parts:
- added C37, C38, C39, C40, C41, C42, C43: GCM188L81H104KA57, GCM188L81H104K57(0.1uF):GCM188L81H104KA57
- added C44, C45: GRM1885C1H102JA01D, GRM1885C1H102JA01D:GRM1885C1H102JA01D
- added JP8: (no value), pinhead:PINHD-1X3
- added Q1: SSM3J332R, SSM3J332R:SSM3J332R
- added R1: 11.8k, CR0603:CR0603
- added R54: 1.2k, CR0603:CR0603
- added R55: 15.8k, CR0603:CR0603
- added R56: 1.6k, CR0603:CR0603
- added R57: 3.3, CR0603:CR0603
- added R58, R59: 1k, CR0603:CR0603
- added R60, R61: 10k, CR0603:CR0603
- added TP1, TP2: GF063PB103K, GF063P B103K:GF063PB103K
Connections:
- new net CS1_OCD1: C44.1, JP8.3, R58.LEFT, U4.OCD1
- new net CS1_OCD2: C45.1, JP8.1, R59.LEFT, U4.OCD2
- new net CS1_REF1: C41.P$2, R1.LEFT, TP1.LEFT, U4.REF1
- new net CS1_REF2: C42.P$2, R55.LEFT, TP2.LEFT, U4.REF2
- new net CURRENT1: C43.P$2, R57.LEFT
- new net N$1: R57.RIGHT, U4.VOUT
- new net N$13: R54.RIGHT, TP1.RIGHT
- new net N$18: Q1.DRAIN, R61.LEFT
- new net N$2: R56.RIGHT, TP2.RIGHT
- new net N$9: JP8.2, Q1.GATE, R60.LEFT
- net +3V3: now also C37.P$2, R1.RIGHT, R55.RIGHT, R58.RIGHT, R59.RIGHT, R61.RIGHT, U4.VDD
- net GND: no longer C3.P$1
- net GND2: now also C3.P$1, C37.P$1, C41.P$1, C42.P$1, C43.P$1, C44.2, C45.2, Q1.SOURCE, R54.LEFT, R56.LEFT, R60.RIGHT, U4.VSS1, U4.VSS2, U6.VSS1, U8.VSS1, U9.VSS1
Other:
- moved on the sheet: U4

Commit message: 電源制御系周り
Parts:
- removed IRLB-1, IRLB-2, IRLB-3, IRLB-4: IRLB3813_2, OKUDA_libraries:IRLB3813_2
- removed SWITCH: 02-JST, con-jst-xh:02-JST
- added C46, C57, C58, C59, C60, C61, C62, C63, C64, C65: GCM188L81H104KA57, GCM188L81H104K57(0.1uF):GCM188L81H104KA57
- added C47, C50, C53, C56: GRM21BC72A105KE01, GRM21BC72A105KE01(1uF):GRM21BC72A105KE01
- added C48, C49, C51, C52, C54, C55: GRM1885C1H102JA01D, GRM1885C1H102JA01D:GRM1885C1H102JA01D
- added INV_SW1, INV_SW2: (no value), pinhead:PINHD-1X2
- added JP10, JP9: (no value), pinhead:PINHD-1X3
- added LED2, LED8: SML-E12V8WT86, SML-E12V8WT86:SML-E12V8WT86
- added Q3, Q4, Q5: SSM3J332R, SSM3J332R:SSM3J332R
- added Q6, Q7: SQJA16EP-T1_GE3, SQJA16EP-T1_GE3:SQJA16EP-T1_GE3
- added Q8: MTB7D0N06RJ3, MTB7D0N06RJ3:MTB7D0N06RJ3
- added R100, R105, R95: 1.2k, CR0603:CR0603
- added R101, R106, R96: 15.8k, CR0603:CR0603
- added R102, R107, R97: 1.6k, CR0603:CR0603
- added R103, R108, R98: 3.3, CR0603:CR0603
- added R104, R67, R99: 11.8k, CR0603:CR0603
- added R109, R111, R112, R77: 1Meg, CR0603:CR0603
- added R110, R115, R63, R66, R70, R73, R76, R80, R83, R88, R91, R94: 10k, CR0603:CR0603
- added R113, R116: 680, CR0603:CR0603
- added R114: 100, CR0603:CR0603
- added R117: 220, CR0603:CR0603
- added R62, R72, R82, R90: 20k, CR0603:CR0603
- added R64, R68, R69, R71, R74, R78, R79, R81, R84, R86, R87, R89, R92: 1k, CR0603:CR0603
- added R65, R75, R85, R93: 2k, CR0603:CR0603
- added SB1, SB2, SB3, SB4: RSX101VAM-30TR, RSX101VAM-30TR:RSX101VAM-30TR
- added SWITCH_1, SWITCH_2: 02-JST, con-jst-xh:02-JST
- added TLP2: TLP152, TLP152:TLP152
- added TP3, TP4, TP5, TP6, TP7, TP8: GF063PB103K, GF063P B103K:GF063PB103K
- added U10, U11, U12, U13: AP331AWG-7, AP331AWG-7:AP331AWG-7
- JP1: device pinhead:PINHD-1X2 -> pinhead:PINHD-1X3
- LED1, LED3: value (none) -> SML-E12V8WT86; device led:LED5MM -> SML-E12V8WT86:SML-E12V8WT86
- R2, R5: device rcl:R-EU_0204/7 -> CR0603:CR0603
- R3: value 1kΩ -> 100; device rcl:R-EU_0204/7 -> CR0603:CR0603
- R4: value 10kΩ -> 10k; device rcl:R-EU_0204/7 -> CR0603:CR0603
- R6: value 1kΩ -> 1k; device rcl:R-EU_0204/7 -> CR0603:CR0603
- R61: value 10k -> 1k
- TLP1: value 2227MC-08-03 -> TLP152; device TLP250H:2227MC-08-03 -> TLP152:TLP152
Connections:
- new net CS2_OCD1: C48.1, JP1.3, R68.LEFT, U6.OCD1
- new net CS2_OCD2: C49.1, JP1.1, R69.LEFT, U6.OCD2
- new net CS2_REF1: C39.P$2, R67.LEFT, TP3.LEFT, U6.REF1
- new net CS2_REF2: C40.P$2, R96.LEFT, TP4.LEFT, U6.REF2
- new net CS3_OCD1: C51.1, JP9.3, R78.LEFT, U8.OCD1
- new net CS3_OCD2: C52.1, JP9.1, R79.LEFT, U8.OCD2
- new net CS3_REF1: C58.P$2, R99.LEFT, TP5.LEFT, U8.REF1
- new net CS3_REF2: C59.P$2, R101.LEFT, TP6.LEFT, U8.REF2
- new net CS4_OCD1: C54.1, JP10.3, R86.LEFT, U9.OCD1
- new net CS4_OCD2: C55.1, JP10.1, R87.LEFT, U9.OCD2
- new net CS4_REF1: C62.P$2, R104.LEFT, TP7.LEFT, U9.REF1
- new net CS4_REF2: C63.P$2, R106.LEFT, TP8.LEFT, U9.REF2
- new net CURRENT2: C46.P$2, R98.LEFT, U1.P9
- new net CURRENT3: C60.P$2, R103.LEFT, U1.P10
- new net CURRENT4: C64.P$2, R108.LEFT, U1.P11
- new net N$100: R105.RIGHT, TP7.RIGHT
- new net N$101: R107.RIGHT, TP8.RIGHT
- new net N$102: R108.RIGHT, U9.VOUT
- new net N$103: R12.LEFT, R20.RIGHT, R33.RIGHT, U7.OUTPUT
- new net N$104: C35.P$1, R46.RIGHT, R47.LEFT
- new net N$106: C47.P$1, R64.LEFT, R65.RIGHT, U10.IN-
- new net N$76: R109.RIGHT, R62.LEFT, R63.RIGHT, U10.IN+
- new net N$77: JP1.2, Q3.GATE, R70.LEFT
- new net N$78: R109.LEFT, R66.RIGHT, SB1.A, U10.OUTPUT
- new net N$79: R95.RIGHT, TP3.RIGHT
- new net N$80: R97.RIGHT, TP4.RIGHT
- new net N$81: R98.RIGHT, U6.VOUT
- new net N$82: R100.RIGHT, TP5.RIGHT
- new net N$83: Q3.DRAIN, R71.LEFT, R74.RIGHT
- new net N$84: R72.LEFT, R73.RIGHT, R77.RIGHT, U11.IN+
- new net N$85: R76.RIGHT, R77.LEFT, SB2.A, U11.OUTPUT
- new net N$86: C50.P$1, R74.LEFT, R75.RIGHT, U11.IN-
- new net N$87: JP9.2, Q4.GATE, R80.LEFT
- new net N$88: Q4.DRAIN, R81.LEFT, R84.RIGHT
- new net N$89: R111.RIGHT, R82.LEFT, R83.RIGHT, U12.IN+
- new net N$90: R110.RIGHT, R111.LEFT, SB3.A, U12.OUTPUT
- new net N$91: C53.P$1, R84.LEFT, R85.RIGHT, U12.IN-
- new net N$92: JP10.2, Q5.GATE, R88.LEFT
- new net N$93: Q5.DRAIN, R89.LEFT, R92.RIGHT
- new net N$94: R112.RIGHT, R90.LEFT, R91.RIGHT, U13.IN+
- new net N$95: R112.LEFT, R94.RIGHT, SB4.A, U13.OUTPUT
- new net N$96: C56.P$1, R92.LEFT, R93.RIGHT, U13.IN-
- new net N$98: R102.RIGHT, TP6.RIGHT
- new net N$99: R103.RIGHT, U8.VOUT
- new net SHUTDOWN: R117.RIGHT, SB1.C, SB2.C, SB3.C, SB4.C
- net +3V3: now also C38.P$2, C57.P$2, C61.P$2, R101.RIGHT, R104.RIGHT, R106.RIGHT, R110.LEFT, R62.RIGHT, R66.LEFT, R67.RIGHT, R68.RIGHT, R69.RIGHT, R71.RIGHT, R72.RIGHT, R76.LEFT, R78.RIGHT, R79.RIGHT, R81.RIGHT, R82.RIGHT, R86.RIGHT, R87.RIGHT, R89.RIGHT, R90.RIGHT, R94.LEFT, R96.RIGHT, R99.RIGHT, U10.VCC, U11.VCC, U12.VCC, U13.VCC, U6.VDD, U8.VDD, U9.VDD
- net CURRENT1: now also U1.P8
- net DEBUG_BT: no longer C35.P$1, R46.RIGHT, R47.LEFT
- net GND: now also C65.P$2, INV_SW2.2, Q6.S, Q7.S, R4.LEFT, SWITCH_2.1, TLP2.GND; no longer IRLB-1.S, IRLB-2.S, IRLB-3.S, IRLB-4.S, JP1.1, R4.2
- net GND2: now also C38.P$1, C39.P$1, C40.P$1, C46.P$1, C47.P$2, C48.2, C49.2, C50.P$2, C51.2, C52.2, C53.P$2, C54.2, C55.2, C56.P$2, C57.P$1, C58.P$1, C59.P$1, C60.P$1, C61.P$1, C62.P$1, C63.P$1, C64.P$1, Q3.SOURCE, Q4.SOURCE, Q5.SOURCE, R100.LEFT, R102.LEFT, R105.LEFT, R107.LEFT, R63.LEFT, R65.LEFT, R70.RIGHT, R73.LEFT, R75.LEFT, R80.RIGHT, R83.LEFT, R85.LEFT, R88.RIGHT, R91.LEFT, R93.LEFT, R95.LEFT, R97.LEFT, TLP2.CATHODE, U10.GND, U11.GND, U12.GND, U13.GND, U6.VSS2, U8.VSS2, U9.VSS2
- net N$11: now also LED8.C, Q8.D, R6.RIGHT; no longer IRLB-2.PD, P-3.P$2, P-4.P$2
- net N$12: now also R114.RIGHT, TLP2.VOUT; no longer IRLB-4.PD, P-7.P$2, P-8.P$2
- net N$14: now also Q8.G, R114.LEFT, R115.RIGHT; no longer EDGE3.P28, EDGE3.P29, EDGE3.P30, EDGE3.P31, EDGE3.P32, EDGE3.P33, EDGE3.P34, EDGE3.P35, EDGE3.P36, EDGE3.P37, EDGE3.P38, EDGE3.P39, P-5.P$1, P-6.P$1
- net N$15: now also CTRL1.2, CTRL2.2, THRU1.2, TLP1.ANODE; no longer IRLB-3.PD, P-5.P$2, P-6.P$2
- net N$16: now also R6.LEFT; no longer R6.2
- net N$17: now also R2.RIGHT; no longer R2.1
- net N$18: now also R64.RIGHT
- net N$19: now also INV_SW1.2, INV_SW2.1, SWITCH_1.1, SWITCH_2.2; no longer CTRL1.2, CTRL2.2, SWITCH.1, THRU1.2, TLP1.ANODE
- net N$20: now also R3.RIGHT; no longer R3.1
- net N$21: now also INV_SW1.1, LED3.C, Q8.S, R115.LEFT, SWITCH_1.2; no longer JP1.2, R6.1
- net N$22: now also Q6.G, Q7.G, R3.LEFT, R4.RIGHT; no longer IRLB-1.G, IRLB-2.G, IRLB-3.G, IRLB-4.G, R3.2, R4.1
- net N$24: now also LED3.A, R113.RIGHT; no longer IRLB-2.D, LED3.C
- net N$25: now also R117.LEFT, TLP2.ANODE; no longer EDGE1.P28, EDGE1.P29, EDGE1.P30, EDGE1.P31, EDGE1.P32, EDGE1.P33, EDGE1.P34, EDGE1.P35, EDGE1.P36, EDGE1.P37, EDGE1.P38, EDGE1.P39, P-1.P$1, P-2.P$1
- net N$26: now also EDGE1.P28, EDGE1.P29, EDGE1.P30, EDGE1.P31, EDGE1.P32, EDGE1.P33, EDGE1.P34, EDGE1.P35, EDGE1.P36, EDGE1.P37, EDGE1.P38, EDGE1.P39, LED2.C, Q6.D; no longer P-3.P$1, P-4.P$1
- net N$3: now also LED2.A, R5.RIGHT; no longer LED3.A, R5.1
- net N$43: no longer R12.LEFT, R20.RIGHT, R33.RIGHT, U7.OUTPUT
- net N$7: now also LED8.A, R116.RIGHT; no longer IRLB-1.PD, P-1.P$2, P-2.P$2
- net N$8: now also EDGE3.P28, EDGE3.P29, EDGE3.P30, EDGE3.P31, EDGE3.P32, EDGE3.P33, EDGE3.P34, EDGE3.P35, EDGE3.P36, EDGE3.P37, EDGE3.P38, EDGE3.P39, Q7.D; no longer P-7.P$1, P-8.P$1
- net VCC: now also C65.P$1, R113.LEFT, R116.LEFT, R2.LEFT, R5.LEFT, TLP2.VCC; no longer R2.2, R5.2, SWITCH.2
Other:
- note added: "タイマ回路の時定数->未決定"
- moved on the sheet: C1, C10, C11, C12, C2, C3, C37, C38, C39, C4, C40, C41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

Commit message: ヒューズ選定
Parts:
- removed P-1, P-2, P-3, P-4, P-5, P-6, P-7, P-8: P-SWITCH, OKUDA_libraries:P-SWITCH
- added FUSE1: FUSEHOLDER-3568, FUSEHOLDER-3568:FUSEHOLDER-3568
- added Q9: BSS138, BSS138:BSS138
- added R118: 220, CR0603:CR0603
- R110: value 10k -> 1Meg
- R111: value 1Meg -> 1k
- R112, R77: value 1Meg -> 10k
- R117: value 220 -> 10k
- R64, R92: value 1k -> 2k
- R66, R76, R88, R94: value 10k -> 1k
- R70, R80: value 10k -> 20k
- R71, R81, R87: value 1k -> 10k
- R72, R82: value 20k -> 2k
- R73, R83: value 10k -> 2k
- R75, R85: value 2k -> 1Meg
Connections:
- removed net N$106: C47.P$1, R64.LEFT, R65.RIGHT, U10.IN-
- removed net N$93: Q5.DRAIN, R89.LEFT, R92.RIGHT
- removed net N$94: R112.RIGHT, R90.LEFT, R91.RIGHT, U13.IN+
- removed net N$95: R112.LEFT, R94.RIGHT, SB4.A, U13.OUTPUT
- removed net N$96: C56.P$1, R92.LEFT, R93.RIGHT, U13.IN-
- new net N$105: C47.P$1, R109.RIGHT, R64.LEFT, R65.RIGHT, U10.IN+
- new net N$97: R62.LEFT, R63.RIGHT, U10.IN-
- net +3V3: now also Q1.SOURCE, Q3.SOURCE, Q4.SOURCE, Q5.SOURCE, R112.LEFT, R118.RIGHT, R60.LEFT, R70.RIGHT, R74.LEFT, R77.LEFT, R80.RIGHT, R84.LEFT, R87.LEFT, R88.RIGHT; no longer R110.LEFT, R61.RIGHT, R71.RIGHT, R72.RIGHT, R76.LEFT, R81.RIGHT, R82.RIGHT, R86.RIGHT, R87.RIGHT
- net CS1_OCD1: now also C48.1, C51.1, C54.1, JP1.3, JP10.3, JP9.3, R68.LEFT, R78.LEFT, R88.LEFT
- net CS1_OCD2: now also C49.1, C52.1, C55.1, JP1.1, JP10.1, JP9.1, R69.LEFT, R79.LEFT, R89.LEFT
- net CS2_OCD1: no longer C48.1, JP1.3, R68.LEFT
- net CS2_OCD2: no longer C49.1, JP1.1, R69.LEFT
- net CS3_OCD1: no longer C51.1, JP9.3, R78.LEFT
- net CS3_OCD2: no longer C52.1, JP9.1, R79.LEFT
- net CS4_OCD1: no longer C54.1, JP10.3, R86.LEFT
- net CS4_OCD2: no longer C55.1, JP10.1, R87.LEFT
- net GND: now also R111.RIGHT, R61.RIGHT, R63.LEFT, R71.LEFT, R76.RIGHT, R81.LEFT, R86.RIGHT, R91.LEFT
- net GND2: now also Q1.DRAIN, Q3.DRAIN, Q4.DRAIN, Q5.DRAIN, Q9.S, R111.LEFT, R117.LEFT, R61.LEFT, R64.RIGHT, R72.RIGHT, R76.LEFT, R82.RIGHT, R86.LEFT, R92.RIGHT; no longer Q1.SOURCE, Q3.SOURCE, Q4.SOURCE, Q5.SOURCE, R60.RIGHT, R63.LEFT, R70.RIGHT, R75.LEFT, R80.RIGHT, R85.LEFT, R88.RIGHT, R91.LEFT
- net N$18: now also JP1.2, Q3.GATE, R77.RIGHT; no longer Q1.DRAIN, R61.LEFT, R64.RIGHT
- net N$25: now also CON1.+, FUSE1.R; no longer R117.LEFT, TLP2.ANODE
- net N$76: now also R74.RIGHT, R75.LEFT, SB2.A, U11.OUTPUT; no longer R109.RIGHT, R62.LEFT, R63.RIGHT, U10.IN+
- net N$77: now also R71.RIGHT, U11.IN-; no longer JP1.2, Q3.GATE
- net N$83: now also C50.P$1, R72.LEFT, R73.RIGHT, R75.RIGHT, U11.IN+; no longer Q3.DRAIN, R71.LEFT, R74.RIGHT
- net N$84: now also JP9.2, Q4.GATE, R87.RIGHT; no longer R72.LEFT, R73.RIGHT, R77.RIGHT, U11.IN+
- net N$85: now also R84.RIGHT, R85.LEFT, SB3.A, U12.OUTPUT; no longer R76.RIGHT, R77.LEFT, SB2.A, U11.OUTPUT
- net N$86: now also R80.LEFT, R81.RIGHT, U12.IN-; no longer C50.P$1, R74.LEFT, R75.RIGHT, U11.IN-
- net N$87: now also C53.P$1, R82.LEFT, R83.RIGHT, R85.RIGHT, U12.IN+; no longer JP9.2, Q4.GATE, R80.LEFT
- net N$88: now also JP10.2, Q5.GATE, R112.RIGHT; no longer Q4.DRAIN, R81.LEFT, R84.RIGHT
- net N$89: now also R110.LEFT, R94.RIGHT, SB4.A, U13.OUTPUT; no longer R111.RIGHT, R82.LEFT, R83.RIGHT, U12.IN+
- net N$9: now also R60.RIGHT; no longer R60.LEFT
- net N$90: now also R90.LEFT, R91.RIGHT, U13.IN-; no longer R110.RIGHT, R111.LEFT, SB3.A, U12.OUTPUT
- net N$91: now also C56.P$1, R110.RIGHT, R92.LEFT, R93.RIGHT, U13.IN+; no longer C53.P$1, R84.LEFT, R85.RIGHT, U12.IN-
- net N$92: now also Q9.D, R118.LEFT, TLP2.ANODE; no longer JP10.2, Q5.GATE, R88.LEFT
- net SHUTDOWN: now also Q9.G
- net VCC: now also FUSE1.L; no longer CON1.+
Other:
- moved on the sheet: C1, C2, C47, C48, C49, C50, C51, C52, C53, C54, C55, C56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

Commit message: kairozunoseiri
Parts:
- removed TLP2: TLP152, TLP152:TLP152
- added C66, C67, C68, C71: GRM21BC72A105KE01, GRM21BC72A105KE01(1uF):GRM21BC72A105KE01
- added C70: GCM188L81H104KA57, GCM188L81H104K57(0.1uF):GCM188L81H104KA57
- added Q10: SQJA16EP-T1_GE3, SQJA16EP-T1_GE3:SQJA16EP-T1_GE3
- added R119, R121: 10k, CR0603:CR0603
- added R120: 1.8k, CR0603:CR0603
- added R122: 300, CR0603:CR0603
- added R123: 270, CR0603:CR0603
- added R124, R125: 10, CR0603:CR0603
- added THRU2: 02-JST, con-jst-xh:02-JST
- added TLP3: TLP152, TLP152:TLP152
- added U14, U15: TCK420G, TCK420G:TCK420G
- added U16, U19: TC7SH00FULJ, TC7SH00FULJ:TC7SH00FULJ
- added U17, U18, U21, U22: TC7S14F, TC7S14F:TC7S14F
- added U20: TLP293, TLP293_Mylib:TLP293
- added ZD1: MMSZ5231B-TP, MMSZ5231B-TP:MMSZ5231B-TP
- added ZD2, ZD3, ZD4, ZD5: MMBZ5248B-TP, MMBZ5248B-TP:MMBZ5248B-TP
- C1: value 50ZLH1000MEFC16X25 -> 50MXG3300MEFCSN22X30; device 50ZLH1000MEFC16X25(1000uF):50ZLH1000MEFC16X25 -> 50MXG3300MEFCSN22X30:50MXG3300MEFCSN22X30
- C2: value GCM188L81H104KA57 -> GRM21BC72A105KE01; device GCM188L81H104K57(0.1uF):GCM188L81H104KA57 -> GRM21BC72A105KE01(1uF):GRM21BC72A105KE01
- R114: value 100 -> 820
- R3: value 100 -> 1
- R4: value 10k -> 220
- R6: value 1k -> 820
Connections:
- net VM1 renamed N$113
- new net 5V1: R121.RIGHT, R123.LEFT, U16.VCC, U17.VCC, U18.VCC, U19.VCC, U21.VCC, ZD1.C
- new net DISABLE: U1.P20, U22.I
- new net EMERGENCY: R120.RIGHT, U14.VCT, U15.VCT, U18.I, U21.O
- new net N$106: R122.LEFT, U19.O
- new net N$107: U16.I0, U18.O
- new net N$108: U16.O, U19.I0, U19.I1
- new net N$109: R121.LEFT, U20.COLLECTOR, U21.I
- new net N$110: R122.RIGHT, TLP3.ANODE
- new net N$111: C66.P$1, C68.P$1, EDGE1.P12, EDGE1.P13, EDGE1.P14, EDGE1.P15, EDGE1.P16, EDGE1.P17, EDGE1.P18, EDGE1.P19, EDGE1.P20, EDGE1.P21, EDGE1.P22, EDGE1.P23, EDGE2.P12, EDGE2.P13, EDGE2.P14, EDGE2.P15, EDGE2.P16, EDGE2.P17, EDGE2.P18, EDGE2.P19, EDGE2.P20, EDGE2.P21, EDGE2.P22, EDGE2.P23, EDGE3.P12, EDGE3.P13, EDGE3.P14, EDGE3.P15, EDGE3.P16, EDGE3.P17, EDGE3.P18, EDGE3.P19, EDGE3.P20, EDGE3.P21, EDGE3.P22, EDGE3.P23, EDGE4.P12, EDGE4.P13, EDGE4.P14, EDGE4.P15, EDGE4.P16, EDGE4.P17, EDGE4.P18, EDGE4.P19, EDGE4.P20, EDGE4.P21, EDGE4.P22, EDGE4.P23, Q6.S, Q7.S, R3.LEFT, R5.LEFT, U14.VOUT, U15.VOUT, ZD2.A, ZD4.A
- new net N$112: Q6.G, R124.LEFT, ZD2.C
- new net N$93: C71.P$1, R120.LEFT, U17.I
- new net N$94: R4.RIGHT, U20.ANODE
- new net N$95: R6.LEFT, TLP3.VOUT
- new net N$96: Q10.G, R119.RIGHT, R6.RIGHT, ZD5.C
- net +3V3: now also U22.VCC
- net GND: now also C66.P$2, C67.P$2, C68.P$2, C70.P$2, C71.P$2, EDGE1.P28, EDGE1.P29, EDGE1.P30, EDGE1.P31, EDGE1.P32, EDGE1.P33, EDGE1.P34, EDGE1.P35, EDGE1.P36, EDGE1.P37, EDGE1.P38, EDGE1.P39, EDGE2.P28, EDGE2.P29, EDGE2.P30, EDGE2.P31, EDGE2.P32, EDGE2.P33, EDGE2.P34, EDGE2.P35, EDGE2.P36, EDGE2.P37, EDGE2.P38, EDGE2.P39, EDGE3.P28, EDGE3.P29, EDGE3.P30, EDGE3.P31, EDGE3.P32, EDGE3.P33, EDGE3.P34, EDGE3.P35, EDGE3.P36, EDGE3.P37, EDGE3.P38, EDGE3.P39, EDGE4.P28, EDGE4.P29, EDGE4.P30, EDGE4.P31, EDGE4.P32, EDGE4.P33, EDGE4.P34, EDGE4.P35, EDGE4.P36, EDGE4.P37, EDGE4.P38, EDGE4.P39, LED2.C, Q10.S, R119.LEFT, TLP3.CATHODE, TLP3.GND, U14.GND, U15.GND, U16.GND, U17.GND, U18.GND, U19.GND, U20.EMITTER, U21.GND, ZD1.A, ZD3.A, ZD5.A; no longer Q6.S, Q7.S, R4.LEFT, TLP2.GND
- net GND2: now also TLP1.CATHODE, U22.GND; no longer TLP2.CATHODE
- net N$11: now also Q10.D, R3.RIGHT; no longer LED8.C, Q8.D, R6.RIGHT
- net N$12: now also TLP1.VOUT; no longer TLP2.VOUT
- net N$14: now also ZD3.C
- net N$15: now also R4.LEFT, THRU2.2; no longer TLP1.ANODE
- net N$16: now also LED8.C, Q8.D, U20.CATHODE; no longer R6.LEFT, TLP1.CATHODE
- net N$20: now also Q7.G, R125.LEFT, ZD4.C; no longer R3.RIGHT, TLP1.VOUT
- net N$21: now also THRU2.1
- net N$22: now also U16.I1, U17.O; no longer Q6.G, Q7.G, R3.LEFT, R4.RIGHT
- net N$26: now also R124.RIGHT, U14.VGATE2; no longer EDGE1.P28, EDGE1.P29, EDGE1.P30, EDGE1.P31, EDGE1.P32, EDGE1.P33, EDGE1.P34, EDGE1.P35, EDGE1.P36, EDGE1.P37, EDGE1.P38, EDGE1.P39, EDGE2.P28, EDGE2.P29, EDGE2.P30, EDGE2.P31, EDGE2.P32, EDGE2.P33, EDGE2.P34, EDGE2.P35, EDGE2.P36, EDGE2.P37, EDGE2.P38, EDGE2.P39, LED2.C, Q6.D
- net N$8: now also R125.RIGHT, U15.VGATE2; no longer EDGE3.P28, EDGE3.P29, EDGE3.P30, EDGE3.P31, EDGE3.P32, EDGE3.P33, EDGE3.P34, EDGE3.P35, EDGE3.P36, EDGE3.P37, EDGE3.P38, EDGE3.P39, EDGE4.P28, EDGE4.P29, EDGE4.P30, EDGE4.P31, EDGE4.P32, EDGE4.P33, EDGE4.P34, EDGE4.P35, EDGE4.P36, EDGE4.P37, EDGE4.P38, EDGE4.P39, Q7.D
- net N$92: now also TLP1.ANODE; no longer TLP2.ANODE
- net SHUTDOWN: now also U22.O
- net VCC: now also C67.P$1, C70.P$1, Q6.D, Q7.D, R123.RIGHT, TLP3.VCC, U14.VIN, U15.VIN; no longer EDGE1.P12, EDGE1.P13, EDGE1.P14, EDGE1.P15, EDGE1.P16, EDGE1.P17, EDGE1.P18, EDGE1.P19, EDGE1.P20, EDGE1.P21, EDGE1.P22, EDGE1.P23, EDGE2.P12, EDGE2.P13, EDGE2.P14, EDGE2.P15, EDGE2.P16, EDGE2.P17, EDGE2.P18, EDGE2.P19, EDGE2.P20, EDGE2.P21, EDGE2.P22, EDGE2.P23, EDGE3.P12, EDGE3.P13, EDGE3.P14, EDGE3.P15, EDGE3.P16, EDGE3.P17, EDGE3.P18, EDGE3.P19, EDGE3.P20, EDGE3.P21, EDGE3.P22, EDGE3.P23, EDGE4.P12, EDGE4.P13, EDGE4.P14, EDGE4.P15, EDGE4.P16, EDGE4.P17, EDGE4.P18, EDGE4.P19, EDGE4.P20, EDGE4.P21, EDGE4.P22, EDGE4.P23, R5.LEFT, TLP2.VCC
Other:
- note added: "Auto Discharger"
- note added: "Battery"
- note added: "Control"
- note added: "Current Sensor"
- note added: "Current Sensor CH1"
- note added: "Current Sensor CH2"
- note added: "Current Sensor CH3"
- note added: "Current Sensor CH4"
- note added: "DeadTime Generator"
- note added: "DeadTime:0.506ms"
- note added: "OCD TIMER"
- note added: "Output"
- note added: "Power Management"
- note added: "USB2.0(Type C)"
- note removed: "BATT input"
- note removed: "control"
- note removed: "output"
- moved on the sheet: B1, BOOTMODE, C10, C11, C12, C13, C14, C15, C16, C17, C18, C19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
