File: src/(Eagle)PowerUnit-Bseries(ver2.0).brd (EAGLE design)
At the start: 100 x 100 mm, 292 parts, among them CON1 XT90PW-M, CON2 XT90PW-F, CON3 XT60PW-F, CON4 XT60PW-F, CON5 XT60PW-F, CON6 XT60PW-F, Q1 SQJA16EP-T1_GE3, Q10 SQJA16EP-T1_GE3, Q11 TMBT3906, Q12 TMBT3906, Q2 SSM3J332R, Q6 SQJA16EP-T1_GE3, SW1 SS-12SDP2, SW2 RDS-16S-1055-SMT-TR, SW3 SSSS213202, SW4 2MS1-T2-B4-M2-Q-E-S, SW5 2MS1-T2-B4-M2-Q-E-S, U1 LQFP64, U10 TC7S14F, U11 MCP6541T-I/LT, U12 MCP6541T-I/LT, U13 TC7S14F, U14 TCK420G, U15 TCKE805NAWSON10B_TOS-REC, U16 TC7SH00FULJ, U17 TC7S14F, U18 TC7S14F, U19 TC7SH00FULJ, U2 MCP2517FD, U20 TLP293, U21 TC7S14F, U22 TC7S14F, U23 TC7S14F, U24 MCP6541T-I/LT, U25 TC7S14F, U26 TC7SH00FULJ, U3 CH340E, U4 CZ-3A04, U5 AP63205WU-7, U6 CZ-3A04, U7 MCP6541T-I/LT, U8 CZ-3A04, U9 CZ-3A04, X1 XRCGB40M000F4M01R0, X2 RH100-24.000-18-1020-EXT-TR, X3 32.768K12.5PI/MC306

Commit message: develop_v2
Parts:
- removed R124: 10, CR0603:CR0603
- removed ZD2: MMBZ5248B-TP, MMBZ5248B-TP:MMBZ5248B-TP
- added LED10, LED9: SML-E12V8WT86, SML-E12V8WT86:SML-E12V8WT86
- added NTC1: NCU15WB473F60RC, NCU15WB473F60RC:NCU15WB473F60RC
- added R79: 680, CR0603:CR0603
- added R80: 33k, CR0603:CR0603
- added R81: 1.8k, CR0603:CR0603
- added R82: 100k, CR0603:CR0603
- added R83: 187k, CR0603:CR0603
- added R84: 0Ω, CR0603:CR0603
- added R85: 100, CR0603:CR0603
- added SB8: RSX101VAM-30TR, RSX101VAM-30TR:RSX101VAM-30TR
- added U27: MCP6541T-I/LT, MCP6541T-I:SC-70-5
- R3: value 1 -> 10; device CR0603:CR0603 -> RSMF2JT10R0:0411V
- R8, R9: value (none) -> 5.1k
- moved R3 270.2 mm to (8.00, 94.0)
- moved SW5 193.1 mm to (-150.0, 38.0)
Connections:
- removed net GND2: B1.3, C10.P$2, C11.P$2, C12.R, C13.P$1, C14.P$2, C15.P$2, C16.2, C17.2, C18.P$2, C19.P$2, C20.P$2, C21.P$2, C22.P$2, C23.P$2, C24.2, C25.P$2, C26.P$2, C27.1, C28.1, C29.1, C3.P$1, C30.1, C31.P$2, C32.P$2, C33.P$2, C34.P$2, C35.P$2, C36.P$2, C37.P$1, C38.P$1, C39.P$1, C4.R, C40.P$1, C41.P$1, C42.P$1, C43.P$1, C44.R, C45.R, C46.P$1, C47.P$2, C48.R, C49.R, C5.R, C50.P$2, C51.R, C52.R, C53.P$2, C54.R, C55.R, C56.P$2, C57.P$1, C58.P$1, C59.P$1, C60.P$1, C61.P$1, C62.P$1, C63.P$1, C64.P$1, C67.P$2, C68.2, C69.P$2, C7.CATHODE, C8.P$2, C9.R, D3.A, GND.1, JP2.1, JP3.1, JP4.1, JP5.1, JP7.1, LED4.K, LED5.K, LED6.K, LED7.K, ML1.11, ML1.5, ML1.7, POW.1, R100.LEFT, R102.LEFT, R105.LEFT, R107.LEFT, R11.RIGHT, R12.LEFT, R15.LEFT, R19.LEFT, R20.LEFT, R22.RIGHT, R29.LEFT, R30.LEFT, R31.LEFT, R37.LEFT, R38.LEFT, R41.LEFT, R45.RIGHT, R49.LEFT, R54.LEFT, R56.LEFT, R61.RIGHT, R66.RIGHT, R72.RIGHT, R75.LEFT, R76.LEFT, R8.LEFT, R9.LEFT, R95.LEFT, R97.LEFT, RJ45_1.2, RJ45_1.8, RJ45_1.LED2_K, RJ45_2.2, RJ45_2.8, RJ45_2.LED2_K, SB6.A, TLP1.CATHODE, TR1.E, TR2.E, U$1.EP, U$1.VSS, U$4.GND, U1.P12, U1.P18, U1.P31, U1.P47, U1.P63, U10.GND, U11.VSS, U12.VSS, U13.GND, U15.GND1, U15.GND2, U15.GND3, U15.GND4, U15.GND5, U2.VSS, U22.GND, U23.GND, U24.VSS, U25.GND, U26.GND, U3.GND, U4.VSS1, U4.VSS2, U5.GND, U6.VSS1, U6.VSS2, U7.VSS, U8.VSS1, U8.VSS2, U9.VSS1, U9.VSS2, USB1.GND1, USB1.GND2, USB1.SHIELD1, USB1.SHIELD2, USB1.SHIELD3, USB1.SHIELD4, X2.2, X2.4
- removed net N$112: Q1.G, Q6.G, R124.LEFT, ZD2.CATHODE
- new net N$120: LED9.A, R79.RIGHT
- new net N$121: R84.RIGHT, U3.RTS#
- new net N$122: R80.RIGHT, R81.LEFT, R83.LEFT, U27.IN+
- new net N$123: R84.LEFT, U3.CTS#
- new net N$124: LED10.A, R85.RIGHT
- new net N$126: R83.RIGHT, R85.LEFT, SB8.A, U27.OUT
- new net PGND: C1.CATHODE, C2.P$2, C65.P$2, C66.P$2, C70.P$2, C71.P$2, CON1.-, CON2.-, EDGE1.P$28, EDGE1.P$29, EDGE1.P$30, EDGE1.P$31, EDGE1.P$32, EDGE1.P$33, EDGE1.P$34, EDGE1.P$35, EDGE1.P$36, EDGE1.P$37, EDGE1.P$38, EDGE1.P$39, EDGE2.P$28, EDGE2.P$29, EDGE2.P$30, EDGE2.P$31, EDGE2.P$32, EDGE2.P$33, EDGE2.P$34, EDGE2.P$35, EDGE2.P$36, EDGE2.P$37, EDGE2.P$38, EDGE2.P$39, EDGE3.P$28, EDGE3.P$29, EDGE3.P$30, EDGE3.P$31, EDGE3.P$32, EDGE3.P$33, EDGE3.P$34, EDGE3.P$35, EDGE3.P$36, EDGE3.P$37, EDGE3.P$38, EDGE3.P$39, EDGE4.P$28, EDGE4.P$29, EDGE4.P$30, EDGE4.P$31, EDGE4.P$32, EDGE4.P$33, EDGE4.P$34, EDGE4.P$35, EDGE4.P$36, EDGE4.P$37, EDGE4.P$38, EDGE4.P$39, GND.2, H1.P$1, H2.P$1, H3.P$1, H4.P$1, INV_SW2.2, LED1.K, LED2.K, LED9.K, Q10.S1, Q10.S2, Q10.S3, R119.LEFT, SW5.O, TLP1.GND, TLP3.CATHODE, TLP3.GND, U14.GND, U16.GND, U17.GND, U18.GND, U19.GND, U20.EMITTER, U21.GND, ZD1.ANODE, ZD5.ANODE
- new net SGND: B1.3, C10.P$2, C11.P$2, C12.R, C13.P$1, C14.P$2, C15.P$2, C16.2, C17.2, C18.P$2, C19.P$2, C20.P$2, C21.P$2, C22.P$2, C23.P$2, C24.2, C25.P$2, C26.P$2, C27.1, C28.1, C29.1, C3.P$1, C30.1, C31.P$2, C32.P$2, C33.P$2, C34.P$2, C35.P$2, C36.P$2, C37.P$1, C38.P$1, C39.P$1, C4.R, C40.P$1, C41.P$1, C42.P$1, C43.P$1, C44.R, C45.R, C46.P$1, C47.P$2, C48.R, C49.R, C5.R, C50.P$2, C51.R, C52.R, C53.P$2, C54.R, C55.R, C56.P$2, C57.P$1, C58.P$1, C59.P$1, C60.P$1, C61.P$1, C62.P$1, C63.P$1, C64.P$1, C67.P$2, C68.2, C69.P$2, C7.CATHODE, C8.P$2, C9.R, D3.A, GND.1, JP2.1, JP3.1, JP4.1, JP5.1, JP7.1, LED10.K, LED4.K, LED5.K, LED6.K, LED7.K, ML1.11, ML1.5, ML1.7, NTC1.L, POW.1, R100.LEFT, R102.LEFT, R105.LEFT, R107.LEFT, R11.RIGHT, R12.LEFT, R15.LEFT, R19.LEFT, R20.LEFT, R22.RIGHT, R29.LEFT, R30.LEFT, R31.LEFT, R37.LEFT, R38.LEFT, R41.LEFT, R45.RIGHT, R49.LEFT, R54.LEFT, R56.LEFT, R61.RIGHT, R66.RIGHT, R72.RIGHT, R75.LEFT, R76.LEFT, R8.LEFT, R81.RIGHT, R9.LEFT, R95.LEFT, R97.LEFT, RJ45_1.2, RJ45_1.8, RJ45_1.LED2_K, RJ45_2.2, RJ45_2.8, RJ45_2.LED2_K, SB6.A, TLP1.CATHODE, TR1.E, TR2.E, U$1.EP, U$1.VSS, U$4.GND, U1.P12, U1.P18, U1.P31, U1.P47, U1.P63, U10.GND, U11.VSS, U12.VSS, U13.GND, U15.GND1, U15.GND2, U15.GND3, U15.GND4, U15.GND5, U2.VSS, U22.GND, U23.GND, U24.VSS, U25.GND, U26.GND, U27.VSS, U3.GND, U4.VSS1, U4.VSS2, U5.GND, U6.VSS1, U6.VSS2, U7.VSS, U8.VSS1, U8.VSS2, U9.VSS1, U9.VSS2, USB1.GND1, USB1.GND2, USB1.SHIELD1, USB1.SHIELD2, USB1.SHIELD3, USB1.SHIELD4, X2.2, X2.4
- new net THERMAL: NTC1.R, R82.RIGHT, U1.P21, U27.IN-
- net +3V3: now also R80.LEFT, R82.LEFT, U27.VDD
- net CS1_OCD1: no longer C48.L, C51.L, C54.L, JP1.3, JP10.3, JP9.3, R24.LEFT, R63.LEFT, R69.LEFT
- net CS1_OCD2: no longer C49.L, C52.L, C55.L, JP1.1, JP10.1, JP9.1, R33.LEFT, R64.LEFT, R70.LEFT
- net CS2_OCD1: now also C48.L, JP1.3, R24.LEFT
- net CS2_OCD2: now also C49.L, JP1.1, R33.LEFT
- net CS3_OCD1: now also C51.L, JP9.3, R63.LEFT
- net CS3_OCD2: now also C52.L, JP9.1, R64.LEFT
- net CS4_OCD1: now also C54.L, JP10.3, R69.LEFT
- net CS4_OCD2: now also C55.L, JP10.1, R70.LEFT
- net GND: no longer C1.CATHODE, C2.P$2, C65.P$2, C66.P$2, C70.P$2, C71.P$2, CON1.-, CON2.-, EDGE1.P$28, EDGE1.P$29, EDGE1.P$30, EDGE1.P$31, EDGE1.P$32, EDGE1.P$33, EDGE1.P$34, EDGE1.P$35, EDGE1.P$36, EDGE1.P$37, EDGE1.P$38, EDGE1.P$39, EDGE2.P$28, EDGE2.P$29, EDGE2.P$30, EDGE2.P$31, EDGE2.P$32, EDGE2.P$33, EDGE2.P$34, EDGE2.P$35, EDGE2.P$36, EDGE2.P$37, EDGE2.P$38, EDGE2.P$39, EDGE3.P$28, EDGE3.P$29, EDGE3.P$30, EDGE3.P$31, EDGE3.P$32, EDGE3.P$33, EDGE3.P$34, EDGE3.P$35, EDGE3.P$36, EDGE3.P$37, EDGE3.P$38, EDGE3.P$39, EDGE4.P$28, EDGE4.P$29, EDGE4.P$30, EDGE4.P$31, EDGE4.P$32, EDGE4.P$33, EDGE4.P$34, EDGE4.P$35, EDGE4.P$36, EDGE4.P$37, EDGE4.P$38, EDGE4.P$39, GND.2, H1.P$1, H2.P$1, H3.P$1, H4.P$1, INV_SW2.2, LED1.K, LED2.K, Q10.S1, Q10.S2, Q10.S3, R119.LEFT, SW5.O, TLP1.GND, TLP3.CATHODE, TLP3.GND, U14.GND, U16.GND, U17.GND, U18.GND, U19.GND, U20.EMITTER, U21.GND, ZD1.ANODE, ZD5.ANODE
- net N$11: now also R3.1; no longer R3.RIGHT
- net N$111: now also R3.2; no longer R3.LEFT, ZD2.ANODE
- net N$25: now also C1.ANODE, R79.LEFT
- net N$26: now also Q1.G, Q6.G; no longer R124.RIGHT
- net SHUTDOWN: now also SB8.C
- net VCC: no longer C1.ANODE

Commit message: 2023/03/07 信号ラインの配線途中
Parts:
- removed C1: 50SEV470M16X16.5, 50SEV470M16X16.5:50SEV470M16X16.5
- removed C25: GCM188L81H104KA57, GCM188L81H104K57(0.1uF):GCM188L81H104KA57
- removed CON6: XT60PW-F, amass:XT60PW-F
- added C72, C73: GCM188L81H104KA57, GCM188L81H104K57(0.1uF):GCM188L81H104KA57
- added D4: GS2M-LTP, GS2M-LTP:GS2M-LTP
- added HEATSINK1: V2020B, V2020B:V2020B
- added IN: XT90PW-M, amass:XT90PW-M
- added JP11: (no value), pinhead:1X06
- added LED11, LED12, LED13, LED14, LED15: SML-E12V8WT86, SML-E12V8WT86:SML-E12V8WT86
- added R86, R87, R89: 150, CR0603:CR0603
- added R88, R90: 100, CR0603:CR0603
- C39, C40, C41, C42, C58, C59, C62, C63: value GCM188L81H104KA57 -> GRM1885C1H102JA01D; device GCM188L81H104K57(0.1uF):GCM188L81H104KA57 -> GRM1885C1H102JA01D:GRM18
- CON1: value XT90PW-M -> XT60PW-F; device amass:XT90PW-M -> amass:XT60PW-F
- CON2: value XT90PW-F -> XT60PW-F; device amass:XT90PW-F -> amass:XT60PW-F
- CON5: value XT60PW-F -> XT90PW-F; device amass:XT60PW-F -> amass:XT90PW-F
- D1, D2: value GS1010FL -> GS2M-LTP; device GS1010FL:GS1010FL -> GS2M-LTP:GS2M-LTP
- INV_SW1, INV_SW2: value (none) -> 02-JST; device pinhead:1X02 -> con-jst-xh:B2B-XH
- R11, R29, R30, R31, R41: value 10k -> 100k
- R113, R116, R2, R5, R79: value 680 -> 1.1k
- R120: value 620 -> 1k
- R32: value 10k -> 10
- R4: value 220 -> 560
- R47, R50: value 10k -> 1k
- R76: value 36k -> 56k
- moved U26 446.8 mm to (101.0, 114.0), flipped to the bottom, turned to 270 degrees
- moved R78 446.3 mm to (97.7, 114.0), flipped to the bottom, turned to 270 degrees
- moved LED10 433.9 mm to (54.0, 103.0), turned to 90 degrees
- moved R85 433.9 mm to (58.0, 103.0), turned to 180 degrees
- moved LED9 429.2 mm to (82.8, 98.0), turned to 90 degrees
- moved R77 428.6 mm to (102.5, 97.0), flipped to the bottom, turned to 270 degrees
- moved R79 427.1 mm to (82.0, 100.0)
- moved TR3 423.5 mm to (98.0, 96.0), flipped to the bottom, turned to 90 degrees
- moved R84 411.4 mm to (93.4, 6.60), turned to 180 degrees
- moved R83 407.6 mm to (27.9, 104.0), turned to 180 degrees
- moved NTC1 406.5 mm to (33.0, 103.0), turned to 270 degrees
- moved SB8 404.0 mm to (26.5, 102.0), turned to 270 degrees
- moved R82 400.1 mm to (33.0, 99.0), turned to 90 degrees
- moved R81 399.2 mm to (31.0, 103.0), turned to 90 degrees
- moved U27 397.8 mm to (28.9, 108.0), turned to 180 degrees
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Connections:
- removed net GND: EDGE1.P$24, EDGE2.P$24, EDGE3.P$24, EDGE4.P$24
- removed net N$15: CTRL1.2, CTRL2.2, R4.LEFT, THRU1.2, THRU2.2
- removed net VCC2: EDGE1.P$27, EDGE2.P$27, EDGE3.P$27, EDGE4.P$27
- new net E5V: C7.ANODE, JP6.3, L1.R, R86.RIGHT, U5.FB
- new net N$112: D4.A, R32.LEFT
- new net N$125: LED11.A, R86.LEFT
- new net N$127: LED15.A, R90.LEFT
- new net N$129: LED13.A, R89.LEFT
- new net N$130: LED14.A, R88.LEFT
- net +3V3: now also C72.P$1, EDGE1.P$27, EDGE2.P$27, EDGE3.P$27, EDGE4.P$27, JP11.1, R88.RIGHT; no longer C25.P$1
- net +5V: now also R89.RIGHT; no longer R32.RIGHT
- net 5V1: now also C73.P$1
- net CS1_REF1: now also C41.L; no longer C41.P$2
- net CS1_REF2: now also C42.L; no longer C42.P$2
- net CS2_REF1: now also C39.L; no longer C39.P$2
- net CS2_REF2: now also C40.L; no longer C40.P$2
- net CS3_REF1: now also C58.L; no longer C58.P$2
- net CS3_REF2: now also C59.L; no longer C59.P$2
- net CS4_REF1: now also C62.L; no longer C62.P$2
- net CS4_REF2: now also C63.L; no longer C63.P$2
- net DISABLE: now also R90.RIGHT
- net IP1: now also CON1.-; no longer CON3.-
- net IP2: now also CON2.-; no longer CON4.-
- net IP3: now also CON3.-; no longer CON5.-
- net IP4: now also CON4.-; no longer CON6.-
- net N$10: now also CON4.+; no longer CON6.+
- net N$103: no longer R32.LEFT
- net N$25: now also IN.+; no longer C1.ANODE, CON1.+
- net N$4: now also CON1.+; no longer CON3.+
- net N$5: now also CON2.+; no longer CON4.+
- net N$55: now also LED12.A, R87.LEFT; no longer C7.ANODE, JP6.3, L1.R, U5.FB
- net N$6: now also CON3.+; no longer CON5.+
- net N$63: now also R49.LEFT; no longer R49.RIGHT
- net N$95: now also D4.C
- net N$96: now also R32.RIGHT
- net NRST: now also JP11.5
- net PGND: now also C73.P$2, CON5.-, IN.-; no longer C1.CATHODE, CON1.-, CON2.-
- net SGND: now also C39.R, C40.R, C41.R, C42.R, C58.R, C59.R, C62.R, C63.R, C72.P$2, EDGE1.P$24, EDGE2.P$24, EDGE3.P$24, EDGE4.P$24, JP11.3, LED11.K, LED12.K, LED13.K, LED14.K, LED15.K, R49.RIGHT; no longer C25.P$2, C39.P$1, C40.P$1, C41.P$1, C42.P$1, C58.P$1, C59.P$1, C62.P$1, C63.P$1, R49.LEFT
- net SWCLK: now also JP11.2
- net SWDIO: now also JP11.4
- net SWO: now also JP11.6
- net U5V: now also R87.RIGHT
- net USART_RX: now also R25.LEFT; no longer R26.LEFT
- net USART_TX: now also R26.LEFT; no longer R25.LEFT
- net VCC: now also CON5.+, CTRL1.2, CTRL2.2, R4.LEFT, THRU1.2, THRU2.2; no longer CON2.+
Routing:
- net EMERGENCY: track 0.00 -> 48.3 mm
- net U5V: track 0.00 -> 43.6 mm
- net VCC: track 0.00 -> 39.8 mm
- net N$96: track 0.00 -> 31.1 mm
- net N$21: track 0.00 -> 28.2 mm
- net N$19: track 0.00 -> 27.3 mm
- net N$111: track 0.00 -> 26.1 mm
- net E5V: track 0.00 -> 23.1 mm
- net SHUTDOWN: track 0.00 -> 17.4 mm
- net N$57: track 0.00 -> 17.4 mm
- net N$45: track 0.00 -> 16.9 mm
- net N$91: track 0.00 -> 15.8 mm
- net DIP_SW3: track 0.00 -> 15.8 mm, vias 0 -> 1
- net N$107: track 0.00 -> 15.1 mm, vias 0 -> 1
- net N$22: track 0.00 -> 13.7 mm, vias 0 -> 1
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- added copper zone on layer 16, net +5V
- added copper zone on layer 16, net IN1
- added copper zone on layer 16, net IN2
- added copper zone on layer 16, net IN3
- added copper zone on layer 16, net IN4
- added copper zone on layer 16, net IP1
- added copper zone on layer 16, net IP2
- added copper zone on layer 16, net IP3
- added copper zone on layer 16, net IP4
- added copper zone on layer 2, net N$10
- added copper zone on layer 1, net N$111
- added copper zone on layer 16, net N$20
- added copper zone on layer 2, net N$25
- added copper zone on layer 2, net N$4
- added copper zone on layer 16, net N$40
- added copper zone on layer 2, net N$5
- added copper zone on layer 2, net N$6
- added copper zone on layer 16, net N$75
- added copper zone on layer 15, net PGND
- added copper zone on layer 1, net U5V
- added copper zone on layer 16, net V+
- added copper zone on layer 1, net VCC
- added copper zone on layer 2, net VCC
Other:
- board size 100 x 100 mm -> 105 x 137 mm

Commit message: 2023/03/08 sintyoku
Parts:
- moved R25 44.9 mm to (101.0, 42.5), flipped to the bottom, turned to 0 degrees
- moved R26 41.5 mm to (101.0, 41.0), flipped to the bottom, turned to 0 degrees
- moved C24 1.08 mm to (81.0, 38.1)
- moved BOOTMODE 0.95 mm to (89.1, 9.14), turned to 270 degrees
- moved C18 0.61 mm to (82.7, 37.5)
- moved C14 0.50 mm to (35.6, 103.5)
- moved C19 0.05 mm to (82.2, 30.5)
- turned C46 to 270 degrees
- turned C60 to 270 degrees
- turned R51 to 180 degrees
Routing:
- net ENC4_B: track 0.00 -> 145.0 mm, vias 0 -> 1
- net ENC3_A: track 0.00 -> 141.7 mm, vias 0 -> 1
- net ENC3_B: track 0.00 -> 141.0 mm, vias 0 -> 1
- net ENC4_A: track 0.00 -> 136.5 mm, vias 0 -> 1
- net N$114: track 0.00 -> 118.2 mm, vias 0 -> 1
- net N$87: track 0.00 -> 110.7 mm, vias 0 -> 1
- net N$83: track 0.00 -> 101.9 mm, vias 0 -> 1
- net SCK: track 0.00 -> 101.8 mm, vias 0 -> 2
- net CS: track 0.00 -> 99.7 mm, vias 0 -> 2
- net MOSI: track 0.00 -> 98.6 mm, vias 0 -> 2
- net MISO: track 0.00 -> 98.3 mm, vias 0 -> 2
- net N$9: track 0.00 -> 92.8 mm, vias 0 -> 1
- net DIR2: track 0.00 -> 90.9 mm, vias 0 -> 1
- net CS1_REF2: track 6.51 -> 86.4 mm, vias 0 -> 2
- net DIR3: track 0.00 -> 78.5 mm
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
Commit message: 2023/03/09進捗分
Parts:
- moved BOOTMODE 6.00 mm to (89.1, 3.14)
- moved C16 1.36 mm to (49.3, 104.6)
- moved U22 0.10 mm to (80.8, 44.1)
Routing:
- net PWM1: track 16.3 -> 183.7 mm
- net ENC1_B: track 0.00 -> 163.2 mm, vias 0 -> 1
- net ENC1_A: track 0.00 -> 162.7 mm, vias 0 -> 1
- net ENC2_B: track 0.00 -> 146.6 mm, vias 0 -> 1
- net ENC2_A: track 0.00 -> 136.3 mm, vias 0 -> 1
- net THERMAL: track 10.0 -> 126.2 mm, vias 0 -> 1
- net DIR1: track 0.00 -> 105.9 mm, vias 0 -> 1
- net DISABLE: track 17.9 -> 115.7 mm, vias 0 -> 2
- net CS1_OCD1: track 7.16 -> 103.0 mm
- net ALIVE_LED: track 0.00 -> 92.1 mm, vias 0 -> 2
- net PWM2: track 0.00 -> 92.1 mm, vias 0 -> 1
- net CS1_OCD2: track 6.84 -> 95.6 mm
- net DEBUG_LED: track 0.00 -> 86.2 mm, vias 0 -> 2
- net COM_LED: track 0.00 -> 81.8 mm, vias 0 -> 2
- net NRST: track 9.22 -> 46.7 mm
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
Commit message: 2023/03/10の進捗
Parts:
- moved H1 158.6 mm to (5.00, 127.0)
- moved H3 158.6 mm to (100.0, 0.00)
- moved C29 1.00 mm to (97.0, 18.5)
- moved C20 0.90 mm to (94.3, 42.0)
- moved R7 0.80 mm to (27.4, 104.3)
- moved SW1 0.80 mm to (23.5, 101.8)
- moved X2 0.50 mm to (85.5, 20.0)
- moved C18 0.14 mm to (82.8, 37.6), turned to 90 degrees
Connections:
- removed net CANH: R7.RIGHT, RJ45_1.3, RJ45_1.4, RJ45_2.3, RJ45_2.4, U$1.CANH
- removed net CANL: RJ45_1.5, RJ45_1.6, RJ45_2.5, RJ45_2.6, SW1.C, U$1.CANL
- new net CAN_H: R7.RIGHT, RJ45_1.5, RJ45_1.6, RJ45_2.5, RJ45_2.6, U$1.CANH
- new net CAN_L: RJ45_1.3, RJ45_1.4, RJ45_2.3, RJ45_2.4, SW1.C, U$1.CANL
- net PGND: no longer H3.P$1, H4.P$1
- net SGND: now also H3.P$1, H4.P$1
Routing:
- net SHUTDOWN: track 17.8 -> 103.4 mm, vias 0 -> 2
- net CAN_H: track 0.00 -> 66.2 mm
- net CAN_L: track 0.00 -> 65.6 mm
- net COM_LED: track 81.8 -> 102.1 mm
- net N$21: track 28.2 -> 44.1 mm
- net N$68: track 0.00 -> 12.0 mm
- net N$65: track 0.00 -> 10.9 mm
- net N$47: track 1.73 -> 7.50 mm
- net N$63: track 0.00 -> 4.76 mm, vias 0 -> 1
- net EMERGENCY: track 48.6 -> 52.3 mm, vias 0 -> 1
- net N$7: track 0.00 -> 3.14 mm
- net N$24: track 0.00 -> 3.14 mm
- net N$23: track 0.00 -> 2.92 mm
- net N$56: track 4.40 -> 6.51 mm
- net +5V: track 12.3 -> 13.8 mm
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- added copper zone on layer 15, net SGND
- added copper zone on layer 16, net SGND

Commit message: 2023/03/20の進捗
Parts:
- moved JP7 0.87 mm to (22.8, 109.5)
- moved R66 0.10 mm to (89.0, 118.0)
- moved R78 0.10 mm to (97.7, 113.9)
Routing:
- net SGND: track 0.00 -> 349.8 mm, vias 0 -> 10
- net +3V3: track 3.10 -> 77.6 mm
- net +5V: track 13.8 -> 73.1 mm
- net 5V1: track 12.5 -> 43.0 mm, vias 0 -> 1
- net PGND: track 0.00 -> 19.3 mm, vias 0 -> 10
- net N$60: track 0.00 -> 11.6 mm, vias 0 -> 1
- net N$127: track 0.00 -> 9.81 mm, vias 0 -> 1
- net N$33: track 0.00 -> 7.77 mm, vias 0 -> 2
- net E5V: track 23.1 -> 29.9 mm
- net N$124: track 0.00 -> 5.31 mm
- net CS2_REF2: track 6.51 -> 10.9 mm
- net N$84: track 0.00 -> 3.42 mm
- net N$125: track 0.00 -> 2.64 mm
- net N$97: track 7.99 -> 9.05 mm, vias 0 -> 2
- net CS1_OCD2: track 95.6 -> 94.7 mm
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- added copper zone on layer 16, net +3V3
- added copper zone on layer 1, net PGND
- added copper zone on layer 1, net SGND

Commit message: 2023/03/21の進捗
Parts:
- moved C28 4.31 mm to (85.0, 23.6), turned to 0 degrees
- moved C37 1.51 mm to (30.6, 18.6), turned to 90 degrees
- moved C61 1.46 mm to (81.6, 18.5), turned to 90 degrees
- moved C57 1.44 mm to (64.5, 18.6), turned to 90 degrees
- moved C38 1.44 mm to (47.5, 18.6), turned to 90 degrees
- moved X2 0.40 mm to (85.8, 20.0)
Routing:
- net +3V3: track 77.6 -> 338.0 mm, vias 0 -> 3
- net CS4_OCD1: track 3.03 -> 163.0 mm, vias 0 -> 2
- net N$21: track 44.1 -> 198.2 mm
- net CS4_OCD2: track 5.56 -> 159.7 mm, vias 0 -> 1
- net SGND: track 349.8 -> 484.2 mm, vias 10 -> 22
- net CS3_REF1: track 6.55 -> 140.3 mm, vias 0 -> 1
- net CS4_REF1: track 13.0 -> 146.7 mm, vias 0 -> 1
- net CS4_REF2: track 10.9 -> 131.8 mm, vias 0 -> 1
- net CS3_REF2: track 10.9 -> 128.9 mm, vias 0 -> 1
- net CS2_REF1: track 12.6 -> 124.6 mm, vias 0 -> 2
- net +5V: track 73.1 -> 173.7 mm, vias 0 -> 1
- net CS1_REF1: track 6.55 -> 105.4 mm, vias 0 -> 2
- net CS3_OCD1: track 7.01 -> 105.4 mm, vias 0 -> 1
- net CS3_OCD2: track 5.48 -> 102.7 mm, vias 0 -> 1
- net CS2_OCD1: track 6.32 -> 100.3 mm, vias 0 -> 1
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
Commit message: 2023/03/23 配線終了
Parts:
- moved C23 0.16 mm to (88.2, 24.6)
- moved R5 0.10 mm to (54.1, 100.0)
- moved C22 0.07 mm to (88.4, 26.0)
Routing:
- net +3V3: track 338.0 -> 695.0 mm, vias 3 -> 26
- net SGND: track 484.2 -> 648.4 mm, vias 22 -> 53
- net N$16: track 4.20 -> 106.6 mm, vias 0 -> 1
- net VCC: track 131.8 -> 204.8 mm, vias 1 -> 3
- net COM_LED: track 102.1 -> 161.7 mm, vias 4 -> 5
- net N$126: track 4.57 -> 59.5 mm
- net 5V1: track 42.9 -> 83.6 mm, vias 1 -> 4
- net +5V: track 173.7 -> 209.1 mm, vias 1 -> 4
- net N$111: track 40.1 -> 65.8 mm, vias 0 -> 2
- net E5V: track 29.9 -> 46.9 mm, vias 0 -> 1
- net PGND: track 41.7 -> 57.5 mm, vias 12 -> 18
- net N$21: track 198.2 -> 208.6 mm, vias 0 -> 1
- net NRST: track 46.7 -> 56.5 mm, vias 0 -> 1
- net N$89: track 0.00 -> 9.35 mm
- net U5V: track 43.7 -> 51.1 mm, vias 0 -> 2
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